Commit message: Torso shell follows the frame: ~13 mm off it, broad shoulders over a slimmer waist
The shell was the convex hull of the whole torso, so the shoulder motors held its sides out
all the way down (up to 44 mm of air). It now follows the frame slice by slice, blending
where the width changes. 39.76 kg with shells; every shell clears all joint ranges.

Co-Authored-By: Claude Opus 5.5 <noreply@anthropic.com>

File: description/urdf/marvin_bot_covers.urdf (robot description, URDF)
Before this commit: robot marvin_bot, 28 links, 27 joints
Links:
- link neck_link: mass 0.16696 -> 0.16495
- link torso_link: mass 9.8666 -> 9.85566
