Commit message: Model: add a wrist bracket so the gripper connects to the forearm
Moves 50 g of the arm structure from each forearm to its wrist link; the
mass budget and standing check are unchanged.

Co-Authored-By: Claude Opus 5.5 <noreply@anthropic.com>

File: description/urdf/marvin_bot.urdf (robot description, URDF)
Before this commit: robot marvin_bot, 28 links, 27 joints
Links:
- link left_forearm_link: mass 0.56 -> 0.51; geometry collision box size=0.07 0.07 0.17; visual box size=0.02 0.06 0.05
- link left_wrist_link: mass 0.0745 -> 0.1245; geometry visual box size=0.05 0.06 0.09; visual cylinder length=0.0248 radius=0.02265
- link right_forearm_link: mass 0.56 -> 0.51; geometry collision box size=0.07 0.07 0.17; visual box size=0.02 0.06 0.05
- link right_wrist_link: mass 0.0745 -> 0.1245; geometry visual box size=0.05 0.06 0.09; visual cylinder length=0.0248 radius=0.02265

Commit message: Static step-up check; ankle dorsiflexion 40° for 17-20 cm stairs
sim/mujoco/check_step_up.py (ported from an earlier prototype, with sideways
weight shift on one foot and a rising rear heel) shows 35° of ankle
dorsiflexion cannot climb 17 cm at any leg length; 38° climbs 20 cm at
0.62-0.69 m hip height. Ankle pitch range is now -40/+40°, hip height
stays 0.65 m. CI runs the 18 cm case.

Co-Authored-By: Claude Opus 5.5 <noreply@anthropic.com>

File: description/urdf/marvin_bot.urdf (robot description, URDF)
Before this commit: robot marvin_bot, 28 links, 27 joints
Joints:
- joint left_ankle_pitch: limit lower=-0.698132 upper=0.610865 effort=72 velocity=50.2655 -> lower=-0.698132 upper=0.698132 effort=72 velocity=50.2655
- joint right_ankle_pitch: limit lower=-0.698132 upper=0.610865 effort=72 velocity=50.2655 -> lower=-0.698132 upper=0.698132 effort=72 velocity=50.2655

Commit message: Ankle linkage design tool; ankles back to RS03
tools/ankle_linkage.py solves the two-crank, two-rod ankle over the full
pitch and roll range and searches its geometry. Best: 45 mm cranks,
~188 mm rods 45 mm behind and 25 mm beside the ankle axis, ratios 1.02
pitch / 0.56 roll. With RS06 the ankle would give only 11 N·m of
continuous roll against ~14 needed on one foot, so the ankles return to
RS03 (mass estimate 37.3 kg). URDF limits use the computed ratios; CI
checks they match the geometry.

Co-Authored-By: Claude Opus 5.5 <noreply@anthropic.com>

File: description/urdf/marvin_bot.urdf (robot description, URDF)
Before this commit: robot marvin_bot, 28 links, 27 joints
Links:
- link left_shin_link: mass 1.792 -> 2.35; geometry collision box size=0.09 0.09 0.22; visual box size=0.02 0.08 0.06
- link right_shin_link: mass 1.792 -> 2.35; geometry collision box size=0.09 0.09 0.22; visual box size=0.02 0.08 0.06
Joints:
- joint left_ankle_pitch: limit lower=-0.698132 upper=0.698132 effort=72 velocity=50.2655 -> lower=-0.698132 upper=0.698132 effort=122.4 velocity=20.02
- joint left_ankle_roll: limit lower=-0.349066 upper=0.349066 effort=43.2 velocity=83.7758 -> lower=-0.349066 upper=0.349066 effort=67.2 velocity=36.4649
- joint right_ankle_pitch: limit lower=-0.698132 upper=0.698132 effort=72 velocity=50.2655 -> lower=-0.698132 upper=0.698132 effort=122.4 velocity=20.02
- joint right_ankle_roll: limit lower=-0.349066 upper=0.349066 effort=43.2 velocity=83.7758 -> lower=-0.349066 upper=0.349066 effort=67.2 velocity=36.4649

Commit message: Ankle layout from real actuator envelopes; vendor CAD fetch script
tools/fetch_vendor_cad.py downloads RobStride's STEP models, pinned to a
commit, into the git-ignored cad/vendor/. Their envelopes (RS03 is
100 mm across, not 106) replace the reseller figures. The two ankle
RS03 now sit side by side 64 mm apart and 125 mm below the knee with
cranks on their outer faces; the linkage search gives 65 mm cranks and
rods +-55 mm aside (ratios 0.86 pitch / 0.83 roll, 31/26 N·m rated at
the worst pose, rod force under 1.3 kN). Foot 110 mm wide. All checks
pass.

Co-Authored-By: Claude Opus 5.5 <noreply@anthropic.com>

File: description/urdf/marvin_bot.urdf (robot description, URDF)
Before this commit: robot marvin_bot, 28 links, 27 joints
Links:
- link left_foot_link: geometry collision box size=0.24 0.11 0.03; visual box size=0.24 0.11 0.03
- link left_forearm_link: geometry collision box size=0.07 0.07 0.17; visual box size=0.02 0.06 0.05
- link left_hip_pitch_link: geometry visual box size=0.08 0.04 0.1; visual cylinder length=0.0557 radius=0.06
- link left_hip_roll_link: geometry visual box size=0.08 0.06 0.1; visual cylinder length=0.0566 radius=0.05
- link left_shin_link: geometry collision box size=0.09 0.09 0.22; visual box size=0.02 0.08 0.06
- link left_shoulder_pitch_link: geometry visual box size=0.06 0.03 0.06; visual cylinder length=0.0566 radius=0.05
- link left_shoulder_roll_link: geometry visual box size=0.06 0.06 0.06; visual cylinder length=0.0505 radius=0.0425
- link left_thigh_link: geometry collision box size=0.09 0.09 0.16; visual box size=0.02 0.08 0.06
- link left_upper_arm_link: geometry collision box size=0.08 0.08 0.14; visual box size=0.07 0.07 0.12
- link pelvis: geometry collision box size=0.14 0.18 0.12; visual box size=0.08 0.12 0.05
- link right_foot_link: geometry collision box size=0.24 0.11 0.03; visual box size=0.24 0.11 0.03
- link right_forearm_link: geometry collision box size=0.07 0.07 0.17; visual box size=0.02 0.06 0.05
- link right_hip_pitch_link: geometry visual box size=0.08 0.04 0.1; visual cylinder length=0.0557 radius=0.06
- link right_hip_roll_link: geometry visual box size=0.08 0.06 0.1; visual cylinder length=0.0566 radius=0.05
- link right_shin_link: geometry collision box size=0.09 0.09 0.22; visual box size=0.02 0.08 0.06
- link right_shoulder_pitch_link: geometry visual box size=0.06 0.03 0.06; visual cylinder length=0.0566 radius=0.05
- link right_shoulder_roll_link: geometry visual box size=0.06 0.06 0.06; visual cylinder length=0.0505 radius=0.0425
- link right_thigh_link: geometry collision box size=0.09 0.09 0.16; visual box size=0.02 0.08 0.06
- link right_upper_arm_link: geometry collision box size=0.08 0.08 0.14; visual box size=0.07 0.07 0.12
- link torso_link: geometry collision box size=0.18 0.26 0.25; visual box size=0.05 0.1 0.06
Joints:
- joint left_ankle_pitch: limit lower=-0.698132 upper=0.698132 effort=122.4 velocity=20.02 -> lower=-0.698132 upper=0.698132 effort=103.2 velocity=23.7446
- joint left_ankle_roll: limit lower=-0.349066 upper=0.349066 effort=67.2 velocity=36.4649 -> lower=-0.349066 upper=0.349066 effort=99.6 velocity=24.6028
- joint right_ankle_pitch: limit lower=-0.698132 upper=0.698132 effort=122.4 velocity=20.02 -> lower=-0.698132 upper=0.698132 effort=103.2 velocity=23.7446
- joint right_ankle_roll: limit lower=-0.349066 upper=0.349066 effort=67.2 velocity=36.4649 -> lower=-0.349066 upper=0.349066 effort=99.6 velocity=24.6028

Commit message: Packaging check; thigh layout, knee 125° and motor positions fixed
tools/check_packaging.py places every motor at its STEP-model size and
every collision box on its link and checks overlaps across the joint
ranges and in combined poses (errors within a limb, warnings between
limbs). Fixes: hip roll RS04 behind the hip pitch RS04; hip yaw joint
40 mm higher on the thigh (roll-yaw 60 mm, yaw-knee 155 mm); knee range
0-125°; shoulder pitch RS03 pulled into the torso; shoulder roll -5°;
neck yaw servo lowered. Step-up, standing and symmetry checks pass;
CI runs the packaging check.

Co-Authored-By: Claude Opus 5.5 <noreply@anthropic.com>

File: description/urdf/marvin_bot.urdf (robot description, URDF)
Before this commit: robot marvin_bot, 28 links, 27 joints
Links:
- link left_shin_link: geometry collision box size=0.09 0.09 0.19; visual box size=0.02 0.08 0.06
- link right_shin_link: geometry collision box size=0.09 0.09 0.19; visual box size=0.02 0.08 0.06
Joints:
- joint left_hip_yaw: origin xyz=0 0 -0.1 -> xyz=0 0 -0.06
- joint left_knee: limit lower=0 upper=2.44346 effort=120 velocity=20.944 -> lower=0 upper=2.18166 effort=120 velocity=20.944; origin xyz=0 0 -0.115 -> xyz=0 0 -0.155
- joint left_shoulder_roll: limit lower=-0.174533 upper=2.0944 effort=60 velocity=20.4204 -> lower=-0.0872665 upper=2.0944 effort=60 velocity=20.4204
- joint right_hip_yaw: origin xyz=0 0 -0.1 -> xyz=0 0 -0.06
- joint right_knee: limit lower=0 upper=2.44346 effort=120 velocity=20.944 -> lower=0 upper=2.18166 effort=120 velocity=20.944; origin xyz=0 0 -0.115 -> xyz=0 0 -0.155
- joint right_shoulder_roll: limit lower=-0.174533 upper=2.0944 effort=60 velocity=20.4204 -> lower=-0.0872665 upper=2.0944 effort=60 velocity=20.4204

Commit message: Leg code-CAD first pass; CAD masses and meshes in the URDF
cad/leg.py draws the legs around the motors at their STEP-model sizes
(hip flange and yoke plates, two-plate hip roll bracket, thigh flange,
side plate and printed shell, shin knee flange, central ankle-motor web
and bearing fork, ankle cross, cranks and rods, foot base, posts, lugs
and TPU sole), pocketed. cad/build.py writes meshes (git-ignored) and
description/cad_model.yaml (mass, CoM, inertia per part) and checks every
part fits the desktop mill or printer; the foot base plates go to a
cutting service. build_urdf.py uses the CAD parts in place of the leg
and foot estimates: 1.72 kg structure + 0.46 kg foot per leg, robot at
37.98 kg, at the 38 kg limit. All checks pass; CI rebuilds the meshes.

Co-Authored-By: Claude Opus 5.5 <noreply@anthropic.com>

File: description/urdf/marvin_bot.urdf (robot description, URDF)
Before this commit: robot marvin_bot, 28 links, 27 joints
Links:
- link left_ankle_link: mass 0.1 -> 0.10925; geometry visual mesh filename=../meshes/left_ankle_cross.stl
- link left_foot_link: mass 0.35 -> 0.4589; geometry collision box size=0.24 0.11 0.03; visual mesh filename=../meshes/left_foot_base.stl
- link left_hip_pitch_link: mass 1.57 -> 1.81643; geometry visual cylinder length=0.0557 radius=0.06; visual mesh filename=../meshes/left_hip_pitch_flange.stl
- link left_hip_roll_link: mass 1.05 -> 1.1097; geometry visual cylinder length=0.0566 radius=0.05; visual mesh filename=../meshes/left_hip_roll_front.stl
- link left_shin_link: mass 2.35 -> 2.47689; geometry collision box size=0.09 0.09 0.19; visual box size=0.02 0.08 0.06
- link left_thigh_link: mass 2.07 -> 1.84937; geometry collision box size=0.09 0.09 0.16; visual box size=0.02 0.08 0.06
- link right_ankle_link: mass 0.1 -> 0.10925; geometry visual mesh filename=../meshes/right_ankle_cross.stl
- link right_foot_link: mass 0.35 -> 0.4589; geometry collision box size=0.24 0.11 0.03; visual mesh filename=../meshes/right_foot_base.stl
- link right_hip_pitch_link: mass 1.57 -> 1.81643; geometry visual cylinder length=0.0557 radius=0.06; visual mesh filename=../meshes/right_hip_pitch_flange.stl
- link right_hip_roll_link: mass 1.05 -> 1.1097; geometry visual cylinder length=0.0566 radius=0.05; visual mesh filename=../meshes/right_hip_roll_front.stl
- link right_shin_link: mass 2.35 -> 2.47689; geometry collision box size=0.09 0.09 0.19; visual box size=0.02 0.08 0.06
- link right_thigh_link: mass 2.07 -> 1.84937; geometry collision box size=0.09 0.09 0.16; visual box size=0.02 0.08 0.06

Commit message: Leg second pass with far-side supports; mass limit 40 kg; stairs note
The second-pass leg (far-side bearings at the knee and hip roll, a
channel-flanged hip block, a ribbed foot) passes cad/strength.py with a
worst safety factor of 2.4, now run in CI. The robot is 39.55 kg; the
computer and battery stay as they are, so the hard limit is raised to
40 kg (target still 35 kg). docs/design/stairs.md documents the stair
climbing status and open issues: knee heat on slow stairs (115% of the
RS04's rating in the static check), the stair policy stopping at the
first step, mass, the knee options, and how they get settled.

Co-Authored-By: Claude Opus 5.5 <noreply@anthropic.com>

File: description/urdf/marvin_bot.urdf (robot description, URDF)
Before this commit: robot marvin_bot, 28 links, 27 joints
Links:
- link left_foot_link: mass 0.4589 -> 0.5876; geometry collision box size=0.24 0.11 0.03; visual mesh filename=../meshes/left_foot_base.stl
- link left_hip_pitch_link: mass 1.81643 -> 2.15698
- link left_hip_roll_link: mass 1.1097 -> 1.28458; geometry visual cylinder length=0.0566 radius=0.05; visual mesh filename=../meshes/left_hip_roll_bar.stl
- link left_shin_link: mass 2.47689 -> 2.59213; geometry collision box size=0.09 0.09 0.19; visual box size=0.02 0.08 0.06
- link left_thigh_link: mass 1.84937 -> 1.87223
- link right_foot_link: mass 0.4589 -> 0.5876; geometry collision box size=0.24 0.11 0.03; visual mesh filename=../meshes/right_foot_base.stl
- link right_hip_pitch_link: mass 1.81643 -> 2.15698
- link right_hip_roll_link: mass 1.1097 -> 1.28458; geometry visual cylinder length=0.0566 radius=0.05; visual mesh filename=../meshes/right_hip_roll_bar.stl
- link right_shin_link: mass 2.47689 -> 2.59213; geometry collision box size=0.09 0.09 0.19; visual box size=0.02 0.08 0.06
- link right_thigh_link: mass 1.84937 -> 1.87223

Commit message: Pelvis and torso CAD, first pass
cad/torso.py draws a pocketed box-frame pelvis (hip pitch RS04s on the
side plates, waist RS03 on top, electronics inside) and a torso of waist
flange, base plate, service-cut uprights carrying the shoulder RS03s, a
neck bridge and a printed chest shell open at the back for the battery.
0.86 + 1.46 kg against 1.0 + 1.8 kg estimated; robot 39.06 kg, stance
knee on a slow 18 cm step at 112% of rated. The pelvis frame is in the
strength check (SF 37). All checks pass.

Co-Authored-By: Claude Opus 5.5 <noreply@anthropic.com>

File: description/urdf/marvin_bot.urdf (robot description, URDF)
Before this commit: robot marvin_bot, 28 links, 27 joints
Links:
- link pelvis: mass 5.24 -> 5.09642; geometry collision box size=0.14 0.18 0.12; visual box size=0.08 0.07 0.05
- link torso_link: mass 9.9745 -> 9.62985; geometry collision box size=0.18 0.26 0.25; visual box size=0.05 0.1 0.05

Commit message: Arm, head and clip-on cover CAD; generated wiring harness
- cad/arm.py: two-plate shoulder brackets (7 mm, SF >= 2.4 in a new hand-load case),
  aluminium motor rings, printed upper-arm and forearm shells, gripper palm and jaw
- cad/head.py: neck bracket, head frame, egg shell, visor with an optics slot, depth camera
- cad/covers.py: optional clip-on covers (offset skins of each link's parts), written only
  into marvin_bot_covers.urdf; the default URDF stays the bare robot
- tools/build_harness.py: per-limb harness routes, service loops, gauges and fuses from the
  CAN map; checked in CI
- mass 39.20 kg bare, 39.76 kg with covers

Co-Authored-By: Claude Opus 5.5 <noreply@anthropic.com>

File: description/urdf/marvin_bot.urdf (robot description, URDF)
Before this commit: robot marvin_bot, 28 links, 27 joints
Links:
- link head_link: mass 0.5 -> 0.35; geometry collision box size=0.15 0.16 0.17; visual mesh filename=../meshes/head_camera.stl
- link left_forearm_link: mass 0.51 -> 0.49661; geometry collision box size=0.07 0.07 0.17; visual box size=0.02 0.06 0.05
- link left_gripper_link: mass 0.2 -> 0.0208; geometry collision box size=0.06 0.08 0.09; visual mesh filename=../meshes/left_gripper_jaw.stl
- link left_shoulder_pitch_link: mass 0.95 -> 1.10425; geometry visual cylinder length=0.0566 radius=0.05; visual mesh filename=../meshes/left_shoulder_back.stl
- link left_shoulder_roll_link: mass 0.671 -> 0.80107; geometry visual cylinder length=0.0505 radius=0.0425; visual mesh filename=../meshes/left_shoulder_roll_front.stl
- link left_upper_arm_link: mass 0.821 -> 0.83251; geometry collision box size=0.08 0.08 0.14; visual cylinder length=0.0505 radius=0.0425
- link left_wrist_link: mass 0.1245 -> 0.14374; geometry visual cylinder length=0.0248 radius=0.02265; visual mesh filename=../meshes/left_gripper_palm.stl
- link neck_link: mass 0.0745 -> 0.11992; geometry visual cylinder length=0.0248 radius=0.02265; visual mesh filename=../meshes/neck_bracket.stl
- link right_forearm_link: mass 0.51 -> 0.49661; geometry collision box size=0.07 0.07 0.17; visual box size=0.02 0.06 0.05
- link right_gripper_link: mass 0.2 -> 0.0208; geometry collision box size=0.06 0.08 0.09; visual mesh filename=../meshes/right_gripper_jaw.stl
- link right_shoulder_pitch_link: mass 0.95 -> 1.10425; geometry visual cylinder length=0.0566 radius=0.05; visual mesh filename=../meshes/right_shoulder_back.stl
- link right_shoulder_roll_link: mass 0.671 -> 0.80107; geometry visual cylinder length=0.0505 radius=0.0425; visual mesh filename=../meshes/right_shoulder_roll_front.stl
- link right_upper_arm_link: mass 0.821 -> 0.83251; geometry collision box size=0.08 0.08 0.14; visual cylinder length=0.0505 radius=0.0425
- link right_wrist_link: mass 0.1245 -> 0.14374; geometry visual cylinder length=0.0248 radius=0.02265; visual mesh filename=../meshes/right_gripper_palm.stl

Commit message: Staggered ankle motors for a slim shin; ring-and-strap plates
- The two ankle RS03 sit one above the other on the shin's centre line between two side
  plates (one under the knee, one behind the ankle): shin ~95 mm wide instead of ~132,
  ankle torque 32 / 25 N·m continuous (pitch / roll), ratios 0.99 / 0.67
- tools/ankle_linkage.py: a position per motor; search over staggered layouts
- Plates reduced to rings on the motors' bolt circles joined by straps (thigh, hip,
  pelvis, torso A-frame uprights, shoulder); all pass cad/strength.py (worst SF 2.2)
- Robot 38.71 kg (was 39.20); 39.30 kg with covers

Co-Authored-By: Claude Opus 5.5 <noreply@anthropic.com>

File: description/urdf/marvin_bot.urdf (robot description, URDF)
Before this commit: robot marvin_bot, 28 links, 27 joints
Links:
- link left_ankle_link: mass 0.10925 -> 0.08558
- link left_hip_pitch_link: mass 2.15698 -> 2.1237
- link left_hip_roll_link: mass 1.28458 -> 1.28059
- link left_shin_link: mass 2.59213 -> 2.64878; geometry collision box size=0.104 0.09 0.097; collision box size=0.11 0.09 0.105
- link left_shoulder_pitch_link: mass 1.10425 -> 1.08805
- link left_shoulder_roll_link: mass 0.80107 -> 0.80432
- link left_thigh_link: mass 1.87223 -> 1.81534
- link pelvis: mass 5.09642 -> 4.984
- link right_ankle_link: mass 0.10925 -> 0.08558
- link right_hip_pitch_link: mass 2.15698 -> 2.1237
- link right_hip_roll_link: mass 1.28458 -> 1.28059
- link right_shin_link: mass 2.59213 -> 2.64878; geometry collision box size=0.104 0.09 0.097; collision box size=0.11 0.09 0.105
- link right_shoulder_pitch_link: mass 1.10425 -> 1.08805
- link right_shoulder_roll_link: mass 0.80107 -> 0.80432
- link right_thigh_link: mass 1.87223 -> 1.81534
- link torso_link: mass 9.62985 -> 9.39763
Joints:
- joint left_ankle_pitch: limit lower=-0.698132 upper=0.698132 effort=103.2 velocity=23.7446 -> lower=-0.698132 upper=0.698132 effort=118.8 velocity=20.6266
- joint left_ankle_roll: limit lower=-0.349066 upper=0.349066 effort=99.6 velocity=24.6028 -> lower=-0.349066 upper=0.349066 effort=80.4 velocity=30.4781
- joint right_ankle_pitch: limit lower=-0.698132 upper=0.698132 effort=103.2 velocity=23.7446 -> lower=-0.698132 upper=0.698132 effort=118.8 velocity=20.6266
- joint right_ankle_roll: limit lower=-0.349066 upper=0.349066 effort=99.6 velocity=24.6028 -> lower=-0.349066 upper=0.349066 effort=80.4 velocity=30.4781

File: description/urdf/marvin_bot_covers.urdf (robot description, URDF)
Before this commit: robot marvin_bot, 28 links, 27 joints
Links:
- link left_ankle_link: mass 0.10925 -> 0.08558
- link left_hip_pitch_link: mass 2.18957 -> 2.15628
- link left_hip_roll_link: mass 1.28458 -> 1.28059
- link left_shin_link: mass 2.65111 -> 2.72151; geometry collision box size=0.104 0.09 0.097; collision box size=0.11 0.09 0.105
- link left_shoulder_pitch_link: mass 1.13992 -> 1.12412
- link left_shoulder_roll_link: mass 0.80107 -> 0.80432
- link left_thigh_link: mass 1.91262 -> 1.8552
- link pelvis: mass 5.1281 -> 5.01568
- link right_ankle_link: mass 0.10925 -> 0.08558
- link right_hip_pitch_link: mass 2.18957 -> 2.15628
- link right_hip_roll_link: mass 1.28458 -> 1.28059
- link right_shin_link: mass 2.65111 -> 2.72151; geometry collision box size=0.104 0.09 0.097; collision box size=0.11 0.09 0.105
- link right_shoulder_pitch_link: mass 1.13992 -> 1.12412
- link right_shoulder_roll_link: mass 0.80107 -> 0.80432
- link right_thigh_link: mass 1.91262 -> 1.8552
- link torso_link: mass 9.82256 -> 9.59403
Joints:
- joint left_ankle_pitch: limit lower=-0.698132 upper=0.698132 effort=103.2 velocity=23.7446 -> lower=-0.698132 upper=0.698132 effort=118.8 velocity=20.6266
- joint left_ankle_roll: limit lower=-0.349066 upper=0.349066 effort=99.6 velocity=24.6028 -> lower=-0.349066 upper=0.349066 effort=80.4 velocity=30.4781
- joint right_ankle_pitch: limit lower=-0.698132 upper=0.698132 effort=103.2 velocity=23.7446 -> lower=-0.698132 upper=0.698132 effort=118.8 velocity=20.6266
- joint right_ankle_roll: limit lower=-0.349066 upper=0.349066 effort=99.6 velocity=24.6028 -> lower=-0.349066 upper=0.349066 effort=80.4 velocity=30.4781
