Commit message: Helmet head and full body shells, with a shell clearance check
- cad/head.py: helmet (hull of crown and chin ellipsoids) with a full-face visor and an
  optics slot; head frame clear of the neck bracket through the pitch range
- cad/covers.py: full shell set as an add-on (torso lofted from rounded sections in eight
  printable pieces with closed sides and shoulder openings, neck sleeve, hip girdle, thigh,
  shin, hip, shoulder, arm sleeves, toe caps), 1.6 mm, 1.10 kg
- python -m cad.covers --check sweeps every joint range plus combined poses and fails on
  any shell contact; in CI
- 38.70 kg bare, 39.80 kg with shells

Co-Authored-By: Claude Opus 5.5 <noreply@anthropic.com>

File: description/urdf/marvin_bot.urdf (robot description, URDF)
Before this commit: robot marvin_bot, 28 links, 27 joints
Links:
- link head_link: mass 0.35 -> 0.3463; geometry collision box size=0.15 0.16 0.162; visual mesh filename=../meshes/head_camera.stl

File: description/urdf/marvin_bot_covers.urdf (robot description, URDF)
Before this commit: robot marvin_bot, 28 links, 27 joints
Links:
- link head_link: mass 0.35 -> 0.3463; geometry collision box size=0.15 0.16 0.162; visual mesh filename=../meshes/head_camera.stl
- link left_foot_link: mass 0.5876 -> 0.61745; geometry collision box size=0.24 0.11 0.03; visual mesh filename=../meshes/left_foot_base.stl
- link left_forearm_link: mass 0.49661 -> 0.52919; geometry collision box size=0.07 0.07 0.17; visual box size=0.02 0.06 0.05
- link left_hip_pitch_link: mass 2.15628 -> 2.14202; geometry visual cylinder length=0.0557 radius=0.06; visual mesh filename=../meshes/left_hip_cover.stl
- link left_shin_link: mass 2.72151 -> 2.71555; geometry collision box size=0.104 0.09 0.097; collision box size=0.11 0.09 0.105
- link left_shoulder_pitch_link: mass 1.12412 -> 1.09903; geometry visual cylinder length=0.0566 radius=0.05; visual mesh filename=../meshes/left_shoulder_back.stl
- link left_thigh_link: mass 1.8552 -> 1.86267
- link left_upper_arm_link: mass 0.83251 -> 0.8491; geometry collision box size=0.08 0.08 0.14; visual cylinder length=0.0505 radius=0.0425
- link neck_link: mass 0.11992 -> 0.14372; geometry visual cylinder length=0.0248 radius=0.02265; visual mesh filename=../meshes/neck_bracket.stl
- link pelvis: mass 5.01568 -> 5.08836; geometry collision box size=0.14 0.18 0.12; visual box size=0.08 0.07 0.05
- link right_foot_link: mass 0.5876 -> 0.61745; geometry collision box size=0.24 0.11 0.03; visual mesh filename=../meshes/right_foot_base.stl
- link right_forearm_link: mass 0.49661 -> 0.52919; geometry collision box size=0.07 0.07 0.17; visual box size=0.02 0.06 0.05
- link right_hip_pitch_link: mass 2.15628 -> 2.14202; geometry visual cylinder length=0.0557 radius=0.06; visual mesh filename=../meshes/right_hip_cover.stl
- link right_shin_link: mass 2.72151 -> 2.71555; geometry collision box size=0.104 0.09 0.097; collision box size=0.11 0.09 0.105
- link right_shoulder_pitch_link: mass 1.12412 -> 1.09903; geometry visual cylinder length=0.0566 radius=0.05; visual mesh filename=../meshes/right_shoulder_back.stl
- link right_thigh_link: mass 1.8552 -> 1.86267
- link right_upper_arm_link: mass 0.83251 -> 0.8491; geometry collision box size=0.08 0.08 0.14; visual cylinder length=0.0505 radius=0.0425
- link torso_link: mass 9.59403 -> 9.92276; geometry collision box size=0.18 0.26 0.25; visual box size=0.05 0.1 0.05

Commit message: More human proportions: shallower torso, helmet head with eye-level camera, longer neck
- Computer stands on edge: torso frame 155 mm deep (was 190); the shell no longer flares
- Helmet head 142 mm wide, 170 mm tall; camera at eye height, half way up the face
- Neck 20 mm longer; torso shell shoulders slope into a collar round a flared neck sleeve;
  upper-arm shell runs down the back of the elbow
- 1.29 m tall, 38.66 kg bare, 39.77 kg with shells; every shell clears through all joint
  ranges

Co-Authored-By: Claude Opus 5.5 <noreply@anthropic.com>

File: description/urdf/marvin_bot.urdf (robot description, URDF)
Before this commit: robot marvin_bot, 28 links, 27 joints
Links:
- link head_link: mass 0.3463 -> 0.33278
- link neck_link: mass 0.11992 -> 0.13288
- link torso_link: mass 9.39763 -> 9.35354; geometry collision box size=0.16 0.26 0.25; visual box size=0.05 0.1 0.05
Joints:
- joint neck_yaw: origin xyz=0 0 0.29 -> xyz=0 0 0.31

File: description/urdf/marvin_bot_covers.urdf (robot description, URDF)
Before this commit: robot marvin_bot, 28 links, 27 joints
Links:
- link head_link: mass 0.3463 -> 0.33278
- link left_upper_arm_link: mass 0.8491 -> 0.85823
- link neck_link: mass 0.14372 -> 0.16696
- link right_upper_arm_link: mass 0.8491 -> 0.85823
- link torso_link: mass 9.92276 -> 9.8666; geometry collision box size=0.16 0.26 0.25; visual box size=0.05 0.1 0.05
Joints:
- joint neck_yaw: origin xyz=0 0 0.29 -> xyz=0 0 0.31

Commit message: Narrower shoulders: arms 158 mm off the centre line (was 188)
- Shoulder pitch motors 30 mm deeper in the torso (centres ±80 mm, joints ±110 mm);
  shoulders 416 mm across (was 476)
- Side frames in two plates: a lower A-frame outside the battery, an upper plate on the
  shoulder motor above the battery and computer, joined by spacers; narrower bays for the
  electronics and keep-alive battery; battery 4.5 mm lower
- Shoulder roll range 0-120° (below 0° the forearm now meets the hip motor)
- 38.80 kg bare, 39.88 kg with shells; packaging, strength and shell checks pass

Co-Authored-By: Claude Opus 5.5 <noreply@anthropic.com>

File: description/urdf/marvin_bot.urdf (robot description, URDF)
Before this commit: robot marvin_bot, 28 links, 27 joints
Links:
- link torso_link: mass 9.35354 -> 9.49306; geometry collision box size=0.16 0.2 0.25; visual box size=0.05 0.08 0.05
Joints:
- joint left_shoulder_pitch: origin xyz=0 0.14 0.25 -> xyz=0 0.11 0.25
- joint left_shoulder_roll: limit lower=-0.0872665 upper=2.0944 effort=60 velocity=20.4204 -> lower=0 upper=2.0944 effort=60 velocity=20.4204
- joint right_shoulder_pitch: origin xyz=0 -0.14 0.25 -> xyz=0 -0.11 0.25
- joint right_shoulder_roll: limit lower=-0.0872665 upper=2.0944 effort=60 velocity=20.4204 -> lower=0 upper=2.0944 effort=60 velocity=20.4204

File: description/urdf/marvin_bot_covers.urdf (robot description, URDF)
Before this commit: robot marvin_bot, 28 links, 27 joints
Links:
- link torso_link: mass 9.85566 -> 9.97174; geometry collision box size=0.16 0.2 0.25; visual box size=0.05 0.08 0.05
Joints:
- joint left_shoulder_pitch: origin xyz=0 0.14 0.25 -> xyz=0 0.11 0.25
- joint left_shoulder_roll: limit lower=-0.0872665 upper=2.0944 effort=60 velocity=20.4204 -> lower=0 upper=2.0944 effort=60 velocity=20.4204
- joint right_shoulder_pitch: origin xyz=0 -0.14 0.25 -> xyz=0 -0.11 0.25
- joint right_shoulder_roll: limit lower=-0.0872665 upper=2.0944 effort=60 velocity=20.4204 -> lower=0 upper=2.0944 effort=60 velocity=20.4204

Commit message: Head profile like a helmet seen from the side; glute and upper-thigh shells
- Head deeper than wide (160 x 142 mm), forward of the neck; visor leaning back 18°;
  underside rising from chin to neck; camera behind a flush tinted window
- Glute shells over the hip roll motors (rounded) and upper-thigh shells over the hip yaw
  motors; shells 1.4 mm; 38.81 kg bare, 39.93 kg with shells; all shells clear

Co-Authored-By: Claude Opus 5.5 <noreply@anthropic.com>

File: description/urdf/marvin_bot.urdf (robot description, URDF)
Before this commit: robot marvin_bot, 28 links, 27 joints
Links:
- link head_link: mass 0.33278 -> 0.34712; geometry collision box size=0.16 0.142 0.158; visual mesh filename=../meshes/head_camera.stl

File: description/urdf/marvin_bot_covers.urdf (robot description, URDF)
Before this commit: robot marvin_bot, 28 links, 27 joints
Links:
- link head_link: mass 0.33278 -> 0.34712; geometry collision box size=0.16 0.142 0.158; visual mesh filename=../meshes/head_camera.stl
- link left_foot_link: mass 0.61745 -> 0.61364
- link left_forearm_link: mass 0.52919 -> 0.52505
- link left_hip_pitch_link: mass 2.14202 -> 2.207; geometry visual cylinder length=0.0557 radius=0.06; visual mesh filename=../meshes/left_glute_cover.stl
- link left_hip_roll_link: mass 1.28059 -> 1.2893; geometry visual cylinder length=0.0566 radius=0.05; visual mesh filename=../meshes/left_hip_roll_bar.stl
- link left_shin_link: mass 2.71555 -> 2.70713
- link left_shoulder_pitch_link: mass 1.09903 -> 1.09768
- link left_thigh_link: mass 1.86267 -> 1.86004
- link left_upper_arm_link: mass 0.85823 -> 0.85497
- link neck_link: mass 0.16495 -> 0.17582
- link pelvis: mass 5.08836 -> 5.07525
- link right_foot_link: mass 0.61745 -> 0.61364
- link right_forearm_link: mass 0.52919 -> 0.52505
- link right_hip_pitch_link: mass 2.14202 -> 2.207; geometry visual cylinder length=0.0557 radius=0.06; visual mesh filename=../meshes/right_glute_cover.stl
- link right_hip_roll_link: mass 1.28059 -> 1.2893; geometry visual cylinder length=0.0566 radius=0.05; visual mesh filename=../meshes/right_hip_roll_bar.stl
- link right_shin_link: mass 2.71555 -> 2.70713
- link right_shoulder_pitch_link: mass 1.09903 -> 1.09768
- link right_thigh_link: mass 1.86267 -> 1.86004
- link right_upper_arm_link: mass 0.85823 -> 0.85497
- link torso_link: mass 9.97174 -> 9.91178

Commit message: Roll-first hip: hip roll motors fixed in the pelvis
- Hip is roll -> pitch -> yaw: roll RS04s on a new pelvis back plate behind the hips; roll
  brackets (U round the roll motor, far-side bearing, outboard bar) carry the pitch RS04s
  at the hip joints; thighs hang from the pitch motors in U-yokes with inner bearings
- Pelvis: back plate, top plate under the waist motor, two gussets, clear of the swinging
  pitch motors; torso 25 mm ahead of the hips (restores 10-20 cm static step-up)
- Ranges: knee 0-130° (was 125°), hip pitch -30-120° (was -40°)
- cad.covers --check also sweeps the real CAD parts against each other; fixes for the
  roll bracket bar, pelvis gussets and the upper-arm shell at full elbow bend
- check_packaging: arm against pelvis is self-collision, like arm against leg
- 38.69 kg bare, 39.78 kg with shells; strength worst SF 2.2

Co-Authored-By: Claude Opus 5.5 <noreply@anthropic.com>

File: description/urdf/marvin_bot.urdf (robot description, URDF)
Before this commit: robot marvin_bot, 28 links, 27 joints
Links:
- link left_hip_pitch_link: mass 2.1237 -> 1.36172; geometry visual cylinder length=0.0566 radius=0.05; visual mesh filename=../meshes/left_hip_pitch_bearing.stl
- link left_hip_roll_link: mass 1.28059 -> 1.87925; geometry visual cylinder length=0.0557 radius=0.06; visual mesh filename=../meshes/left_hip_roll_bar.stl
- link left_upper_arm_link: mass 0.83251 -> 0.80462
- link pelvis: mass 4.984 -> 5.24774; geometry collision box size=0.09 0.13 0.13; collision box size=0.09 0.13 0.13
- link right_hip_pitch_link: mass 2.1237 -> 1.36172; geometry visual cylinder length=0.0566 radius=0.05; visual mesh filename=../meshes/right_hip_pitch_bearing.stl
- link right_hip_roll_link: mass 1.28059 -> 1.87925; geometry visual cylinder length=0.0557 radius=0.06; visual mesh filename=../meshes/right_hip_roll_bar.stl
- link right_upper_arm_link: mass 0.83251 -> 0.80462
Joints:
- joint left_hip_pitch: limit lower=-0.698132 upper=2.0944 effort=120 velocity=20.944 -> lower=-0.523599 upper=2.0944 effort=120 velocity=20.944; origin xyz=0 0.075 0 -> xyz=0 -0.025 0; parent pelvis -> left_hip_roll_link
- joint left_hip_roll: origin xyz=0 0.025 -0.085 -> xyz=0 0.1 0; parent left_hip_pitch_link -> pelvis
- joint left_hip_yaw: origin xyz=0 0 -0.06 -> xyz=0 0.025 -0.145; parent left_hip_roll_link -> left_hip_pitch_link
- joint left_knee: limit lower=0 upper=2.18166 effort=120 velocity=20.944 -> lower=0 upper=2.26893 effort=120 velocity=20.944
- joint right_hip_pitch: limit lower=-0.698132 upper=2.0944 effort=120 velocity=20.944 -> lower=-0.523599 upper=2.0944 effort=120 velocity=20.944; origin xyz=0 -0.075 0 -> xyz=0 0.025 0; parent pelvis -> right_hip_roll_link
- joint right_hip_roll: origin xyz=0 -0.025 -0.085 -> xyz=0 -0.1 0; parent right_hip_pitch_link -> pelvis
- joint right_hip_yaw: origin xyz=0 0 -0.06 -> xyz=0 -0.025 -0.145; parent right_hip_roll_link -> right_hip_pitch_link
- joint right_knee: limit lower=0 upper=2.18166 effort=120 velocity=20.944 -> lower=0 upper=2.26893 effort=120 velocity=20.944
- joint waist_yaw: origin xyz=0 0 0.115 -> xyz=0.025 0 0.115

File: description/urdf/marvin_bot_covers.urdf (robot description, URDF)
Before this commit: robot marvin_bot, 28 links, 27 joints
Links:
- link left_hip_pitch_link: mass 2.207 -> 1.39598; geometry visual cylinder length=0.0566 radius=0.05; visual mesh filename=../meshes/left_hip_pitch_bearing.stl
- link left_hip_roll_link: mass 1.2893 -> 1.94504; geometry visual cylinder length=0.0557 radius=0.06; visual mesh filename=../meshes/left_glute_cover.stl
- link left_upper_arm_link: mass 0.85497 -> 0.827
- link pelvis: mass 5.07525 -> 5.29587; geometry collision box size=0.09 0.13 0.13; collision box size=0.09 0.13 0.13
- link right_hip_pitch_link: mass 2.207 -> 1.39598; geometry visual cylinder length=0.0566 radius=0.05; visual mesh filename=../meshes/right_hip_pitch_bearing.stl
- link right_hip_roll_link: mass 1.2893 -> 1.94504; geometry visual cylinder length=0.0557 radius=0.06; visual mesh filename=../meshes/right_glute_cover.stl
- link right_upper_arm_link: mass 0.85497 -> 0.827
Joints:
- joint left_hip_pitch: limit lower=-0.698132 upper=2.0944 effort=120 velocity=20.944 -> lower=-0.523599 upper=2.0944 effort=120 velocity=20.944; origin xyz=0 0.075 0 -> xyz=0 -0.025 0; parent pelvis -> left_hip_roll_link
- joint left_hip_roll: origin xyz=0 0.025 -0.085 -> xyz=0 0.1 0; parent left_hip_pitch_link -> pelvis
- joint left_hip_yaw: origin xyz=0 0 -0.06 -> xyz=0 0.025 -0.145; parent left_hip_roll_link -> left_hip_pitch_link
- joint left_knee: limit lower=0 upper=2.18166 effort=120 velocity=20.944 -> lower=0 upper=2.26893 effort=120 velocity=20.944
- joint right_hip_pitch: limit lower=-0.698132 upper=2.0944 effort=120 velocity=20.944 -> lower=-0.523599 upper=2.0944 effort=120 velocity=20.944; origin xyz=0 -0.075 0 -> xyz=0 0.025 0; parent pelvis -> right_hip_roll_link
- joint right_hip_roll: origin xyz=0 -0.025 -0.085 -> xyz=0 -0.1 0; parent right_hip_pitch_link -> pelvis
- joint right_hip_yaw: origin xyz=0 0 -0.06 -> xyz=0 -0.025 -0.145; parent right_hip_roll_link -> right_hip_pitch_link
- joint right_knee: limit lower=0 upper=2.18166 effort=120 velocity=20.944 -> lower=0 upper=2.26893 effort=120 velocity=20.944
- joint waist_yaw: origin xyz=0 0 0.115 -> xyz=0.025 0 0.115

Commit message: Box thigh top round the hip pitch motor; roll bracket bars over the roll motors
- Thigh top is a closed box (outer and inner walls, front and back walls, yaw motor under
  its floor) instead of a U of two plates; outer wall 6 mm (was 8), SF 5.6
- Roll bracket bars run over the roll motors; pelvis back plate full width only below the
  roll axes with a narrow spine above, clear of the bars at 45° roll
- No shells over the hip roll motors
- 38.78 kg bare, 39.74 kg with shells; part and shell sweep, packaging, stairs pass

Co-Authored-By: Claude Opus 5.5 <noreply@anthropic.com>

File: description/urdf/marvin_bot.urdf (robot description, URDF)
Before this commit: robot marvin_bot, 28 links, 27 joints
Links:
- link left_hip_pitch_link: mass 1.36172 -> 1.40563; geometry visual cylinder length=0.0566 radius=0.05; visual mesh filename=../meshes/left_hip_pitch_back.stl
- link left_hip_roll_link: mass 1.87925 -> 1.87796
- link pelvis: mass 5.24774 -> 5.2486
- link right_hip_pitch_link: mass 1.36172 -> 1.40563; geometry visual cylinder length=0.0566 radius=0.05; visual mesh filename=../meshes/right_hip_pitch_back.stl
- link right_hip_roll_link: mass 1.87925 -> 1.87796

File: description/urdf/marvin_bot_covers.urdf (robot description, URDF)
Before this commit: robot marvin_bot, 28 links, 27 joints
Links:
- link left_hip_pitch_link: mass 1.39598 -> 1.43993; geometry visual cylinder length=0.0566 radius=0.05; visual mesh filename=../meshes/left_hip_pitch_back.stl
- link left_hip_roll_link: mass 1.94504 -> 1.87796; geometry visual cylinder length=0.0557 radius=0.06; visual mesh filename=../meshes/left_hip_roll_bar.stl
- link pelvis: mass 5.29587 -> 5.29761
- link right_hip_pitch_link: mass 1.39598 -> 1.43993; geometry visual cylinder length=0.0566 radius=0.05; visual mesh filename=../meshes/right_hip_pitch_back.stl
- link right_hip_roll_link: mass 1.94504 -> 1.87796; geometry visual cylinder length=0.0557 radius=0.06; visual mesh filename=../meshes/right_hip_roll_bar.stl
