Commit message: Real actuator outlines and mounts; servos the right way up; computer mount
- actuators.yaml: body, rear driver cap and hole circles from RobStride's drawings and STEP
  models; robot.yaml: each motor's output direction (and servo case direction)
- build_urdf: stepped motor outlines (body + cap, servo boxes) in visuals, packaging and sweep
- cad/mounts.py: rear rings on the real stator holes with cap clearance, posts to the outer
  plates (now light spiders where they carry no bolts), output flanges with the output hole
  circle and a running relief; every leg, pelvis, torso and arm mount reworked
- Neck bracket, head frame, neck sleeve and gripper rebuilt round the servos' real axis
- Computer on edge, fan forward (chest vents), ports to the sides, on a plate behind it;
  H-shaped neck bridge clear of the shoulder motor caps
- 39.12 kg bare, 39.94 kg with 1.2 mm shells; strength, packaging and sweep pass

Co-Authored-By: Claude Opus 5.5 <noreply@anthropic.com>

File: description/urdf/marvin_bot.urdf (robot description, URDF)
Before this commit: robot marvin_bot, 28 links, 27 joints
Links:
- link head_link: mass 0.34712 -> 0.35031
- link left_forearm_link: mass 0.49661 -> 0.48156
- link left_gripper_link: mass 0.0208 -> 0.02297
- link left_hip_pitch_link: mass 1.40563 -> 1.44808; geometry visual cylinder length=0.0125 radius=0.039; visual cylinder length=0.0441 radius=0.05
- link left_hip_roll_link: mass 1.87796 -> 1.86304; geometry visual cylinder length=0.0132 radius=0.047; visual cylinder length=0.0425 radius=0.06
- link left_shin_link: mass 2.64878 -> 2.75449; geometry collision box size=0.104 0.09 0.097; collision box size=0.11 0.09 0.105
- link left_shoulder_pitch_link: mass 1.08805 -> 1.15244; geometry visual cylinder length=0.0125 radius=0.039; visual cylinder length=0.0441 radius=0.05
- link left_shoulder_roll_link: mass 0.80432 -> 0.83212; geometry visual cylinder length=0.014 radius=0.035; visual cylinder length=0.0365 radius=0.0425
- link left_thigh_link: mass 1.81534 -> 1.79985; geometry collision box size=0.09 0.09 0.16; visual box size=0.02 0.08 0.06
- link left_upper_arm_link: mass 0.80462 -> 0.76797; geometry collision box size=0.08 0.08 0.14; visual cylinder length=0.014 radius=0.035
- link left_wrist_link: mass 0.14374 -> 0.14572; geometry visual box size=0.0248 0.0358 0.0453; visual mesh filename=../meshes/left_gripper_palm.stl
- link neck_link: mass 0.13288 -> 0.15905; geometry visual box size=0.0248 0.0358 0.0453; visual mesh filename=../meshes/neck_bracket.stl
- link pelvis: mass 5.2486 -> 5.26377; geometry collision box size=0.09 0.13 0.13; collision box size=0.09 0.13 0.13
- link right_forearm_link: mass 0.49661 -> 0.48156
- link right_gripper_link: mass 0.0208 -> 0.02297
- link right_hip_pitch_link: mass 1.40563 -> 1.44808; geometry visual cylinder length=0.0125 radius=0.039; visual cylinder length=0.0441 radius=0.05
- link right_hip_roll_link: mass 1.87796 -> 1.86304; geometry visual cylinder length=0.0132 radius=0.047; visual cylinder length=0.0425 radius=0.06
- link right_shin_link: mass 2.64878 -> 2.75449; geometry collision box size=0.104 0.09 0.097; collision box size=0.11 0.09 0.105
- link right_shoulder_pitch_link: mass 1.08805 -> 1.15244; geometry visual cylinder length=0.0125 radius=0.039; visual cylinder length=0.0441 radius=0.05
- link right_shoulder_roll_link: mass 0.80432 -> 0.83212; geometry visual cylinder length=0.014 radius=0.035; visual cylinder length=0.0365 radius=0.0425
- link right_thigh_link: mass 1.81534 -> 1.79985; geometry collision box size=0.09 0.09 0.16; visual box size=0.02 0.08 0.06
- link right_upper_arm_link: mass 0.80462 -> 0.76797; geometry collision box size=0.08 0.08 0.14; visual cylinder length=0.014 radius=0.035
- link right_wrist_link: mass 0.14374 -> 0.14572; geometry visual box size=0.0248 0.0358 0.0453; visual mesh filename=../meshes/right_gripper_palm.stl
- link torso_link: mass 9.49306 -> 9.45915; geometry collision box size=0.16 0.2 0.25; visual box size=0.0453 0.0248 0.0358

File: description/urdf/marvin_bot_covers.urdf (robot description, URDF)
Before this commit: robot marvin_bot, 28 links, 27 joints
Links:
- link head_link: mass 0.34712 -> 0.35031
- link left_foot_link: mass 0.61364 -> 0.60986
- link left_forearm_link: mass 0.52505 -> 0.50587
- link left_gripper_link: mass 0.0208 -> 0.02297
- link left_hip_pitch_link: mass 1.43993 -> 1.47745; geometry visual cylinder length=0.0125 radius=0.039; visual cylinder length=0.0441 radius=0.05
- link left_hip_roll_link: mass 1.87796 -> 1.86304; geometry visual cylinder length=0.0132 radius=0.047; visual cylinder length=0.0425 radius=0.06
- link left_shin_link: mass 2.70713 -> 2.80533; geometry collision box size=0.104 0.09 0.097; collision box size=0.11 0.09 0.105
- link left_shoulder_pitch_link: mass 1.09768 -> 1.16036; geometry visual cylinder length=0.0125 radius=0.039; visual cylinder length=0.0441 radius=0.05
- link left_shoulder_roll_link: mass 0.80432 -> 0.83212; geometry visual cylinder length=0.014 radius=0.035; visual cylinder length=0.0365 radius=0.0425
- link left_thigh_link: mass 1.86004 -> 1.83796; geometry collision box size=0.09 0.09 0.16; visual box size=0.02 0.08 0.06
- link left_upper_arm_link: mass 0.827 -> 0.7871; geometry collision box size=0.08 0.08 0.14; visual cylinder length=0.014 radius=0.035
- link left_wrist_link: mass 0.14374 -> 0.14572; geometry visual box size=0.0248 0.0358 0.0453; visual mesh filename=../meshes/left_gripper_palm.stl
- link neck_link: mass 0.17582 -> 0.19965; geometry visual box size=0.0248 0.0358 0.0453; visual mesh filename=../meshes/neck_bracket.stl
- link pelvis: mass 5.29761 -> 5.30601; geometry collision box size=0.09 0.13 0.13; collision box size=0.09 0.13 0.13
- link right_foot_link: mass 0.61364 -> 0.60986
- link right_forearm_link: mass 0.52505 -> 0.50587
- link right_gripper_link: mass 0.0208 -> 0.02297
- link right_hip_pitch_link: mass 1.43993 -> 1.47745; geometry visual cylinder length=0.0125 radius=0.039; visual cylinder length=0.0441 radius=0.05
- link right_hip_roll_link: mass 1.87796 -> 1.86304; geometry visual cylinder length=0.0132 radius=0.047; visual cylinder length=0.0425 radius=0.06
- link right_shin_link: mass 2.70713 -> 2.80533; geometry collision box size=0.104 0.09 0.097; collision box size=0.11 0.09 0.105
- link right_shoulder_pitch_link: mass 1.09768 -> 1.16036; geometry visual cylinder length=0.0125 radius=0.039; visual cylinder length=0.0441 radius=0.05
- link right_shoulder_roll_link: mass 0.80432 -> 0.83212; geometry visual cylinder length=0.014 radius=0.035; visual cylinder length=0.0365 radius=0.0425
- link right_thigh_link: mass 1.86004 -> 1.83796; geometry collision box size=0.09 0.09 0.16; visual box size=0.02 0.08 0.06
- link right_upper_arm_link: mass 0.827 -> 0.7871; geometry collision box size=0.08 0.08 0.14; visual cylinder length=0.014 radius=0.035
- link right_wrist_link: mass 0.14374 -> 0.14572; geometry visual box size=0.0248 0.0358 0.0453; visual mesh filename=../meshes/right_gripper_palm.stl
- link torso_link: mass 9.91178 -> 9.81819; geometry collision box size=0.16 0.2 0.25; visual box size=0.0453 0.0248 0.0358

Commit message: Electronics bay, battery cradle and limb-root bulkheads
Lay out the bought electronics at typical outlines in the torso and pelvis
(cad/electrical.py), with the battery slide-out cradle, printed guides and
latch, and a power and signal bulkhead per limb. The harness names each
limb's bulkhead and the clip pair for every service loop, and the leg chain
follows the roll-first order. Printed parts are strength-checked and the
ankle linkage is in the part sweep. BOM: compact 12 V servo DC-DC, limb
connectors. 39.13 kg bare, 39.96 kg with shells.

Co-Authored-By: Claude Opus 5.5 <noreply@anthropic.com>

File: description/urdf/marvin_bot.urdf (robot description, URDF)
Before this commit: robot marvin_bot, 28 links, 27 joints
Links:
- link left_upper_arm_link: mass 0.76797 -> 0.78954
- link pelvis: mass 5.26377 -> 5.33377; geometry collision box size=0.09 0.13 0.13; collision box size=0.09 0.13 0.13
- link right_upper_arm_link: mass 0.76797 -> 0.78954
- link torso_link: mass 9.45915 -> 9.36338; geometry collision box size=0.16 0.2 0.25; visual box size=0.0453 0.0248 0.0358

File: description/urdf/marvin_bot_covers.urdf (robot description, URDF)
Before this commit: robot marvin_bot, 28 links, 27 joints
Links:
- link left_upper_arm_link: mass 0.7871 -> 0.80874
- link pelvis: mass 5.30601 -> 5.37601; geometry collision box size=0.09 0.13 0.13; collision box size=0.09 0.13 0.13
- link right_upper_arm_link: mass 0.7871 -> 0.80874
- link torso_link: mass 9.81819 -> 9.72242; geometry collision box size=0.16 0.2 0.25; visual box size=0.0453 0.0248 0.0358

Commit message: Four-finger hands on a wrist pitch joint; mass limit includes the shells
Replaces the 1-DOF grippers with the two bought 8-servo hand kits. The
gripper STS3250 becomes a wrist pitch joint (+-60 deg) in a printed cradle
under the wrist RS00, with a printed U and plate carrying the hand
(modelled as its envelope, 0.40 kg each). The forearm is 0.188 m to the
wrist axis, a person's at this height. 27 body DOF.

The hard limit now applies to the robot with hands and body shells and is
41 kg (39.86 kg bare, 40.68 kg with shells). Harness, BOM (hands, 5 V
converters, a serial adapter per hand), strength and sweep checks, Isaac
Lab gains and the motion scripts follow. Also includes the retargeting
changes behind the third tracker (leg and torso scaling, standing rest
pose, torso keypoint frame).

Co-Authored-By: Claude Opus 5.5 <noreply@anthropic.com>

File: description/urdf/marvin_bot.urdf (robot description, URDF)
Before this commit: robot marvin_bot, 28 links, 27 joints
Links:
- removed link left_gripper_link
- removed link right_gripper_link
- added link left_palm_link, mass 0.41656; collision box size=0.05 0.11 0.16; visual mesh filename=../meshes/left_hand.stl
- added link right_palm_link, mass 0.41656; collision box size=0.05 0.11 0.16; visual mesh filename=../meshes/right_hand.stl
- link left_wrist_link: mass 0.14572 -> 0.11534; geometry collision box size=0.035 0.05 0.05; visual box size=0.0248 0.0358 0.0453
- link right_wrist_link: mass 0.14572 -> 0.11534; geometry collision box size=0.035 0.05 0.05; visual box size=0.0248 0.0358 0.0453
Joints:
- removed joint left_gripper
- removed joint right_gripper
- added joint left_wrist_pitch: type revolute, parent left_wrist_link, child left_palm_link, origin xyz=0 0 -0.063, axis 0 -1 0, limit lower=-1.0472 upper=1.0472 effort=4.9 velocity=7.85398
- added joint right_wrist_pitch: type revolute, parent right_wrist_link, child right_palm_link, origin xyz=0 0 -0.063, axis 0 -1 0, limit lower=-1.0472 upper=1.0472 effort=4.9 velocity=7.85398

File: description/urdf/marvin_bot_covers.urdf (robot description, URDF)
Before this commit: robot marvin_bot, 28 links, 27 joints
Links:
- removed link left_gripper_link
- removed link right_gripper_link
- added link left_palm_link, mass 0.41656; collision box size=0.05 0.11 0.16; visual mesh filename=../meshes/left_hand.stl
- added link right_palm_link, mass 0.41656; collision box size=0.05 0.11 0.16; visual mesh filename=../meshes/right_hand.stl
- link left_wrist_link: mass 0.14572 -> 0.11534; geometry collision box size=0.035 0.05 0.05; visual box size=0.0248 0.0358 0.0453
- link right_wrist_link: mass 0.14572 -> 0.11534; geometry collision box size=0.035 0.05 0.05; visual box size=0.0248 0.0358 0.0453
Joints:
- removed joint left_gripper
- removed joint right_gripper
- added joint left_wrist_pitch: type revolute, parent left_wrist_link, child left_palm_link, origin xyz=0 0 -0.063, axis 0 -1 0, limit lower=-1.0472 upper=1.0472 effort=4.9 velocity=7.85398
- added joint right_wrist_pitch: type revolute, parent right_wrist_link, child right_palm_link, origin xyz=0 0 -0.063, axis 0 -1 0, limit lower=-1.0472 upper=1.0472 effort=4.9 velocity=7.85398

Commit message: Real AmazingHand meshes on the wrists; docs and credits audit
The hands are now the AmazingHand (Pollen Robotics) meshes, derived from
its CC-BY-4.0 CAD and MuJoCo models by tools/build_hand_mesh.py and kept
under their own licence in description/third_party/amazing_hand/ with
attribution. Real left and right hands; the mount plate takes the hand's
6 x M3 on a 42 mm circle. README render updated.

Docs: README goals (6-DOF arms, hand payload), 40 kg mass in the safety
notes, payload requirement note, third-party licence rules in
CONTRIBUTING.md, and credits for the CAD libraries, the Orin model, the
hand servos, the body-proportion source and Kimodo's licences.

Co-Authored-By: Claude Opus 5.5 <noreply@anthropic.com>

File: description/urdf/marvin_bot.urdf (robot description, URDF)
Before this commit: robot marvin_bot, 28 links, 27 joints
Links:
- link left_palm_link: mass 0.41656 -> 0.41829
- link right_palm_link: mass 0.41656 -> 0.41829

File: description/urdf/marvin_bot_covers.urdf (robot description, URDF)
Before this commit: robot marvin_bot, 28 links, 27 joints
Links:
- link left_palm_link: mass 0.41656 -> 0.41829
- link right_palm_link: mass 0.41656 -> 0.41829

Commit message: Wider shoulder yaw, hip roll, hip yaw and waist yaw ranges
Motion tracking showed the narrow ranges limiting skills (the two-hand
wave and reach held the shoulder yaw on its 90 deg stop; sidesteps hit
the -20 deg hip roll). Four ranges widen with no part, mass or cost
change: shoulder yaw +-150 (was +-90), hip roll -30 (was -20), hip yaw
+-90 (was +-45), waist yaw +-150 (was +-90). The clearance checks pass;
the new contacts are between limbs and avoided by control. URDFs and
harness service loops regenerated. Shoulder roll below 0 needs a
pitch-dependent limit and is not changed here.

Co-Authored-By: Claude Opus 5.5 <noreply@anthropic.com>

File: description/urdf/marvin_bot.urdf (robot description, URDF)
Before this commit: robot marvin_bot, 28 links, 27 joints
Joints:
- joint left_hip_roll: limit lower=-0.349066 upper=0.785398 effort=120 velocity=20.944 -> lower=-0.523599 upper=0.785398 effort=120 velocity=20.944
- joint left_hip_yaw: limit lower=-0.785398 upper=0.785398 effort=60 velocity=20.4204 -> lower=-1.5708 upper=1.5708 effort=60 velocity=20.4204
- joint left_shoulder_yaw: limit lower=-1.5708 upper=1.5708 effort=36 velocity=50.2655 -> lower=-2.61799 upper=2.61799 effort=36 velocity=50.2655
- joint right_hip_roll: limit lower=-0.349066 upper=0.785398 effort=120 velocity=20.944 -> lower=-0.523599 upper=0.785398 effort=120 velocity=20.944
- joint right_hip_yaw: limit lower=-0.785398 upper=0.785398 effort=60 velocity=20.4204 -> lower=-1.5708 upper=1.5708 effort=60 velocity=20.4204
- joint right_shoulder_yaw: limit lower=-1.5708 upper=1.5708 effort=36 velocity=50.2655 -> lower=-2.61799 upper=2.61799 effort=36 velocity=50.2655
- joint waist_yaw: limit lower=-1.5708 upper=1.5708 effort=60 velocity=20.4204 -> lower=-2.61799 upper=2.61799 effort=60 velocity=20.4204

File: description/urdf/marvin_bot_covers.urdf (robot description, URDF)
Before this commit: robot marvin_bot, 28 links, 27 joints
Joints:
- joint left_hip_roll: limit lower=-0.349066 upper=0.785398 effort=120 velocity=20.944 -> lower=-0.523599 upper=0.785398 effort=120 velocity=20.944
- joint left_hip_yaw: limit lower=-0.785398 upper=0.785398 effort=60 velocity=20.4204 -> lower=-1.5708 upper=1.5708 effort=60 velocity=20.4204
- joint left_shoulder_yaw: limit lower=-1.5708 upper=1.5708 effort=36 velocity=50.2655 -> lower=-2.61799 upper=2.61799 effort=36 velocity=50.2655
- joint right_hip_roll: limit lower=-0.349066 upper=0.785398 effort=120 velocity=20.944 -> lower=-0.523599 upper=0.785398 effort=120 velocity=20.944
- joint right_hip_yaw: limit lower=-0.785398 upper=0.785398 effort=60 velocity=20.4204 -> lower=-1.5708 upper=1.5708 effort=60 velocity=20.4204
- joint right_shoulder_yaw: limit lower=-1.5708 upper=1.5708 effort=36 velocity=50.2655 -> lower=-2.61799 upper=2.61799 effort=36 velocity=50.2655
- joint waist_yaw: limit lower=-1.5708 upper=1.5708 effort=60 velocity=20.4204 -> lower=-2.61799 upper=2.61799 effort=60 velocity=20.4204

Commit message: Honest mass budget; stronger thigh plate, thinner shin and pelvis plates
The mass budget now carries the weighed computer (0.877 kg, was a 1.5 kg
estimate) and the fasteners (0.4 kg) and limb harness (0.5 kg) the CAD
leaves out: 40.74 kg with shells, under the 41 kg limit.

The thigh plate, weak against a sideways fall onto the knee (finite
elements: SF 0.5 at an estimated 1 x body weight), is now 9 mm stock
pocketed to a 2 mm floor (lighten(..., floor=)): SF 2.3 in the new side
case in cad/strength.py, +61 g a side. The shin side plates go 6 -> 4 mm
and the pelvis back plate 8 -> 6 mm (SF 2.1 each). The torso base, which
a hand catch twists, needs FEA and is recorded as open.

Co-Authored-By: Claude Opus 5.5 <noreply@anthropic.com>

File: description/urdf/marvin_bot.urdf (robot description, URDF)
Before this commit: robot marvin_bot, 28 links, 27 joints
Links:
- link left_forearm_link: mass 0.48156 -> 0.52156; geometry collision box size=0.07 0.07 0.17; visual box size=0.02 0.03 0.1
- link left_hip_roll_link: mass 1.86304 -> 1.8617
- link left_shin_link: mass 2.75449 -> 2.7412; geometry collision box size=0.104 0.09 0.097; collision box size=0.11 0.09 0.105
- link left_thigh_link: mass 1.79985 -> 2.00031; geometry collision box size=0.09 0.09 0.16; visual box size=0.02 0.04 0.16
- link left_upper_arm_link: mass 0.78954 -> 0.86954; geometry collision box size=0.08 0.08 0.14; visual box size=0.02 0.03 0.12
- link pelvis: mass 5.33377 -> 5.3131; geometry collision box size=0.09 0.13 0.13; collision box size=0.09 0.13 0.13
- link right_forearm_link: mass 0.48156 -> 0.52156; geometry collision box size=0.07 0.07 0.17; visual box size=0.02 0.03 0.1
- link right_hip_roll_link: mass 1.86304 -> 1.8617
- link right_shin_link: mass 2.75449 -> 2.7412; geometry collision box size=0.104 0.09 0.097; collision box size=0.11 0.09 0.105
- link right_thigh_link: mass 1.79985 -> 2.00031; geometry collision box size=0.09 0.09 0.16; visual box size=0.02 0.04 0.16
- link right_upper_arm_link: mass 0.78954 -> 0.86954; geometry collision box size=0.08 0.08 0.14; visual box size=0.02 0.03 0.12
- link torso_link: mass 9.36338 -> 8.82038; geometry collision box size=0.16 0.2 0.25; visual box size=0.0453 0.0248 0.0358

File: description/urdf/marvin_bot_covers.urdf (robot description, URDF)
Before this commit: robot marvin_bot, 28 links, 27 joints
Links:
- link left_forearm_link: mass 0.50587 -> 0.54587; geometry collision box size=0.07 0.07 0.17; visual box size=0.02 0.03 0.1
- link left_hip_roll_link: mass 1.86304 -> 1.8617
- link left_shin_link: mass 2.80533 -> 2.79161; geometry collision box size=0.104 0.09 0.097; collision box size=0.11 0.09 0.105
- link left_thigh_link: mass 1.83796 -> 2.03853; geometry collision box size=0.09 0.09 0.16; visual box size=0.02 0.04 0.16
- link left_upper_arm_link: mass 0.80874 -> 0.88874; geometry collision box size=0.08 0.08 0.14; visual box size=0.02 0.03 0.12
- link pelvis: mass 5.37601 -> 5.35506; geometry collision box size=0.09 0.13 0.13; collision box size=0.09 0.13 0.13
- link right_forearm_link: mass 0.50587 -> 0.54587; geometry collision box size=0.07 0.07 0.17; visual box size=0.02 0.03 0.1
- link right_hip_roll_link: mass 1.86304 -> 1.8617
- link right_shin_link: mass 2.80533 -> 2.79161; geometry collision box size=0.104 0.09 0.097; collision box size=0.11 0.09 0.105
- link right_thigh_link: mass 1.83796 -> 2.03853; geometry collision box size=0.09 0.09 0.16; visual box size=0.02 0.04 0.16
- link right_upper_arm_link: mass 0.80874 -> 0.88874; geometry collision box size=0.08 0.08 0.14; visual box size=0.02 0.03 0.12
- link torso_link: mass 9.72242 -> 9.17942; geometry collision box size=0.16 0.2 0.25; visual box size=0.0453 0.0248 0.0358

Commit message: Fastener and harness mass boxes not drawn; README robot picture updated
The fastener and limb-harness budget items added with the honest mass
budget are boxes spread over each link (for mass and inertia), and the
URDF builder drew them like the computer and battery boxes: a grey box
over the chest and dark boxes over the pelvis and legs. They are now
left out of the visuals (NOT_DRAWN in tools/build_urdf.py); masses and
inertias are unchanged (39.91 kg bare, 40.74 kg with shells).
docs/media/robot.webp is re-rendered with the current plates.

Co-Authored-By: Claude Opus 5.5 <noreply@anthropic.com>

File: description/urdf/marvin_bot.urdf (robot description, URDF)
Before this commit: robot marvin_bot, 28 links, 27 joints
Links:
- link left_forearm_link: geometry collision box size=0.07 0.07 0.17; visual box size=0.02 0.06 0.05
- link left_shin_link: geometry collision box size=0.104 0.09 0.097; collision box size=0.11 0.09 0.105
- link left_thigh_link: geometry collision box size=0.09 0.09 0.16; visual box size=0.02 0.08 0.06
- link left_upper_arm_link: geometry collision box size=0.08 0.08 0.14; visual cylinder length=0.014 radius=0.035
- link pelvis: geometry collision box size=0.09 0.13 0.13; collision box size=0.09 0.13 0.13
- link right_forearm_link: geometry collision box size=0.07 0.07 0.17; visual box size=0.02 0.06 0.05
- link right_shin_link: geometry collision box size=0.104 0.09 0.097; collision box size=0.11 0.09 0.105
- link right_thigh_link: geometry collision box size=0.09 0.09 0.16; visual box size=0.02 0.08 0.06
- link right_upper_arm_link: geometry collision box size=0.08 0.08 0.14; visual cylinder length=0.014 radius=0.035
- link torso_link: geometry collision box size=0.16 0.2 0.25; visual box size=0.0453 0.0248 0.0358

File: description/urdf/marvin_bot_covers.urdf (robot description, URDF)
Before this commit: robot marvin_bot, 28 links, 27 joints
Links:
- link left_forearm_link: geometry collision box size=0.07 0.07 0.17; visual box size=0.02 0.06 0.05
- link left_shin_link: geometry collision box size=0.104 0.09 0.097; collision box size=0.11 0.09 0.105
- link left_thigh_link: geometry collision box size=0.09 0.09 0.16; visual box size=0.02 0.08 0.06
- link left_upper_arm_link: geometry collision box size=0.08 0.08 0.14; visual cylinder length=0.014 radius=0.035
- link pelvis: geometry collision box size=0.09 0.13 0.13; collision box size=0.09 0.13 0.13
- link right_forearm_link: geometry collision box size=0.07 0.07 0.17; visual box size=0.02 0.06 0.05
- link right_shin_link: geometry collision box size=0.104 0.09 0.097; collision box size=0.11 0.09 0.105
- link right_thigh_link: geometry collision box size=0.09 0.09 0.16; visual box size=0.02 0.08 0.06
- link right_upper_arm_link: geometry collision box size=0.08 0.08 0.14; visual cylinder length=0.014 radius=0.035
- link torso_link: geometry collision box size=0.16 0.2 0.25; visual box size=0.0453 0.0248 0.0358
