Commit message: Depth camera level with the face in a light printed frame
The camera window behind the curved face let through about a third of
the depth camera's view. The camera now sits with its front level with
the face's front on the centre line, in a light printed frame like a
pair of spectacles across the black visor, so nothing is ahead of its
lenses (a ray cast clears 100% of the 90 x 65 deg view). The frame is
only the part outside the helmet (22 g); the camera slides in from the
front and screws to a new arm on the head frame by its tripod thread.
The head is 17 g heavier (0.452 kg); the robot 40.75 kg with shells.

The camera's outline, lens positions and tripod thread are measured
from Orbbec's mesh and URDF (OrbbecSDK_ROS2, Apache-2.0), which
tools/fetch_vendor_cad.py now downloads, pinned to a commit, into the
git-ignored cad/vendor/. Credited in ACKNOWLEDGMENTS.md.

Co-Authored-By: Claude Opus 5.5 <noreply@anthropic.com>

File: description/urdf/marvin_bot.urdf (robot description, URDF)
Before this commit: robot marvin_bot, 28 links, 27 joints
Links:
- link head_link: mass 0.35031 -> 0.36741; geometry collision box size=0.16 0.142 0.158; visual mesh filename=../meshes/head_camera.stl

File: description/urdf/marvin_bot_covers.urdf (robot description, URDF)
Before this commit: robot marvin_bot, 28 links, 27 joints
Links:
- link head_link: mass 0.35031 -> 0.36741; geometry collision box size=0.16 0.142 0.158; visual mesh filename=../meshes/head_camera.stl

Commit message: Longer torso and legs (1.44 m), battery high for a V-shaped torso; 42 kg limit
At 1.29 m the hands hung almost to the knees. The torso is 100 mm
longer, the shoulder roll joint 25 mm closer under the shoulder pitch
joint, and the legs 50 mm longer (thigh above the hip yaw motor, so the
thigh plate still fits the mill; shin with the ankle motors kept at the
ankle). Fingertips reach 0.556 m (a person's 0.542 m), hips 0.48 of the
height. The battery sits high on a shelf under the shoulder motors and
the lower frames lean in to the computer's width, so the torso narrows
to 160 mm at the waist (was 188). Shin straps 44 mm (SF 2.3); chest
shell in two prints, torso cover seams at 200 mm.

40.41 kg bare, 41.38 kg with shells; limit now 42 kg. Static stair
check: knee 118% of rated (was 109%), hip roll 105%. Policies must be
retrained on the new model.

Co-Authored-By: Claude Opus 5.5 <noreply@anthropic.com>

File: description/urdf/marvin_bot.urdf (robot description, URDF)
Before this commit: robot marvin_bot, 28 links, 27 joints
Links:
- link left_hip_pitch_link: mass 1.44808 -> 1.51381
- link left_shin_link: mass 2.7412 -> 2.77964
- link left_shoulder_pitch_link: mass 1.15244 -> 1.12998
- link right_hip_pitch_link: mass 1.44808 -> 1.51381
- link right_shin_link: mass 2.7412 -> 2.77964
- link right_shoulder_pitch_link: mass 1.15244 -> 1.12998
- link torso_link: mass 8.82038 -> 9.14397; geometry collision box size=0.16 0.2 0.25; visual box size=0.0453 0.0248 0.0358
Joints:
- joint left_ankle_pitch: origin xyz=0 0 -0.29 -> xyz=0 0 -0.315
- joint left_hip_yaw: origin xyz=0 0.025 -0.145 -> xyz=0 0.025 -0.17
- joint left_shoulder_pitch: origin xyz=0 0.11 0.25 -> xyz=0 0.11 0.35
- joint left_shoulder_roll: origin xyz=0 0.048 -0.05 -> xyz=0 0.048 -0.025
- joint neck_yaw: origin xyz=0 0 0.31 -> xyz=0 0 0.41
- joint right_ankle_pitch: origin xyz=0 0 -0.29 -> xyz=0 0 -0.315
- joint right_hip_yaw: origin xyz=0 -0.025 -0.145 -> xyz=0 -0.025 -0.17
- joint right_shoulder_pitch: origin xyz=0 -0.11 0.25 -> xyz=0 -0.11 0.35
- joint right_shoulder_roll: origin xyz=0 -0.048 -0.05 -> xyz=0 -0.048 -0.025

File: description/urdf/marvin_bot_covers.urdf (robot description, URDF)
Before this commit: robot marvin_bot, 28 links, 27 joints
Links:
- link left_hip_pitch_link: mass 1.47745 -> 1.54966
- link left_shin_link: mass 2.79161 -> 2.83858
- link left_shoulder_pitch_link: mass 1.16036 -> 1.13716
- link right_hip_pitch_link: mass 1.47745 -> 1.54966
- link right_shin_link: mass 2.79161 -> 2.83858
- link right_shoulder_pitch_link: mass 1.16036 -> 1.13716
- link torso_link: mass 9.17942 -> 9.61363; geometry collision box size=0.16 0.2 0.25; visual box size=0.0453 0.0248 0.0358
Joints:
- joint left_ankle_pitch: origin xyz=0 0 -0.29 -> xyz=0 0 -0.315
- joint left_hip_yaw: origin xyz=0 0.025 -0.145 -> xyz=0 0.025 -0.17
- joint left_shoulder_pitch: origin xyz=0 0.11 0.25 -> xyz=0 0.11 0.35
- joint left_shoulder_roll: origin xyz=0 0.048 -0.05 -> xyz=0 0.048 -0.025
- joint neck_yaw: origin xyz=0 0 0.31 -> xyz=0 0 0.41
- joint right_ankle_pitch: origin xyz=0 0 -0.29 -> xyz=0 0 -0.315
- joint right_hip_yaw: origin xyz=0 -0.025 -0.145 -> xyz=0 -0.025 -0.17
- joint right_shoulder_pitch: origin xyz=0 -0.11 0.25 -> xyz=0 -0.11 0.35
- joint right_shoulder_roll: origin xyz=0 -0.048 -0.05 -> xyz=0 -0.048 -0.025

Commit message: Shoe-shaped foot plate with a slight V toe
The foot plate and sole were rectangles. They now follow a shoe's outline: full-width heel with rounded corners, widest at the ball, and a toe narrowing in a slight V to a rounded point set towards the inside; the toe cap follows. A 20 mm rib down the middle of the toe keeps a toe-first landing at SF 3.3. Feet -67 g; simulation keeps its rectangular contact box.

Co-Authored-By: Claude Opus 5.5 <noreply@anthropic.com>

File: description/urdf/marvin_bot.urdf (robot description, URDF)
Before this commit: robot marvin_bot, 28 links, 27 joints
Links:
- link left_foot_link: mass 0.5876 -> 0.55411; geometry collision box size=0.24 0.11 0.03; visual mesh filename=../meshes/left_foot_base.stl
- link right_foot_link: mass 0.5876 -> 0.55411; geometry collision box size=0.24 0.11 0.03; visual mesh filename=../meshes/right_foot_base.stl

File: description/urdf/marvin_bot_covers.urdf (robot description, URDF)
Before this commit: robot marvin_bot, 28 links, 27 joints
Links:
- link left_foot_link: mass 0.60986 -> 0.57162; geometry collision box size=0.24 0.11 0.03; visual mesh filename=../meshes/left_foot_base.stl
- link right_foot_link: mass 0.60986 -> 0.57162; geometry collision box size=0.24 0.11 0.03; visual mesh filename=../meshes/right_foot_base.stl

Commit message: Shoulder roll below 0° with the arm forward (coupled limit)
Shoulder roll goes to -10° with the arm 45-75° forward and -20° at 90-135°, and stays at 0° with
the arm hanging, so the clap, reach and squat references can bring the hands to the middle.
coupled_limits in robot.yaml; cad.covers --check and check_packaging.py check every point of it.
-30° was checked and needs the shoulder rebuilt. check_robot.py runs the delayed DC motors in
Isaac Lab's Python actuator path, as the tasks do.

Co-Authored-By: Claude Opus 5.5 <noreply@anthropic.com>

File: description/urdf/marvin_bot.urdf (robot description, URDF)
Before this commit: robot marvin_bot, 28 links, 27 joints
Joints:
- joint left_shoulder_roll: limit lower=0 upper=2.0944 effort=60 velocity=20.4204 -> lower=-0.349066 upper=2.0944 effort=60 velocity=20.4204
- joint right_shoulder_roll: limit lower=0 upper=2.0944 effort=60 velocity=20.4204 -> lower=-0.349066 upper=2.0944 effort=60 velocity=20.4204

File: description/urdf/marvin_bot_covers.urdf (robot description, URDF)
Before this commit: robot marvin_bot, 28 links, 27 joints
Joints:
- joint left_shoulder_roll: limit lower=0 upper=2.0944 effort=60 velocity=20.4204 -> lower=-0.349066 upper=2.0944 effort=60 velocity=20.4204
- joint right_shoulder_roll: limit lower=0 upper=2.0944 effort=60 velocity=20.4204 -> lower=-0.349066 upper=2.0944 effort=60 velocity=20.4204

Commit message: CAD: lighten with 7075, isogrid pockets, bolt pads and printed parts; pelvis passes
Strength-limited plates go to 7075 (hip roll web and front plate, thigh plate and ribs, shin
plates and bridge, the pelvis, torso base, bridge and shoulder plates, shoulder brackets, foot
base); parts with margin are thinner; plates under a motor keep only a pad round each stator
bolt; the hip roll strip, battery shelf and neck bracket are printed PA-CF. The shin bridge moves
out and grows (SF 1.2 -> 6.7); the pelvis gets fillets and solid zones at the waist (worst SF 3.1).
Mass budget synced to the CAD: 41.59 kg bare, 42.52 kg with shells (0.52 kg over the limit).

Still open: shoulder pitch bracket SF 2.0-2.1 (layout), printed arm shells SF 0.3.

Co-Authored-By: Claude Opus 5.5 <noreply@anthropic.com>

File: description/urdf/marvin_bot.urdf (robot description, URDF)
Before this commit: robot marvin_bot, 28 links, 27 joints
Links:
- link left_ankle_link: mass 0.08558 -> 0.04888
- link left_foot_link: mass 0.55411 -> 0.4149
- link left_forearm_link: mass 0.52156 -> 0.51981
- link left_hip_pitch_link: mass 1.51381 -> 1.50236
- link left_hip_roll_link: mass 1.8617 -> 1.96168; geometry visual cylinder length=0.0132 radius=0.047; visual cylinder length=0.0425 radius=0.06
- link left_shin_link: mass 2.77964 -> 2.89625; geometry collision box size=0.104 0.09 0.097; collision box size=0.11 0.09 0.105
- link left_shoulder_pitch_link: mass 1.12998 -> 1.16922
- link left_shoulder_roll_link: mass 0.83212 -> 0.83559
- link left_thigh_link: mass 2.00031 -> 2.02313; geometry collision box size=0.09 0.09 0.16; visual box size=0.02 0.08 0.06
- link left_upper_arm_link: mass 0.86954 -> 0.88431
- link neck_link: mass 0.15905 -> 0.11085
- link pelvis: mass 5.3131 -> 6.38544; geometry collision box size=0.09 0.13 0.13; collision box size=0.09 0.13 0.13
- link right_ankle_link: mass 0.08558 -> 0.04888
- link right_foot_link: mass 0.55411 -> 0.4149
- link right_forearm_link: mass 0.52156 -> 0.51981
- link right_hip_pitch_link: mass 1.51381 -> 1.50236
- link right_hip_roll_link: mass 1.8617 -> 1.96168; geometry visual cylinder length=0.0132 radius=0.047; visual cylinder length=0.0425 radius=0.06
- link right_shin_link: mass 2.77964 -> 2.89625; geometry collision box size=0.104 0.09 0.097; collision box size=0.11 0.09 0.105
- link right_shoulder_pitch_link: mass 1.12998 -> 1.16922
- link right_shoulder_roll_link: mass 0.83212 -> 0.83559
- link right_thigh_link: mass 2.00031 -> 2.02313; geometry collision box size=0.09 0.09 0.16; visual box size=0.02 0.08 0.06
- link right_upper_arm_link: mass 0.86954 -> 0.88431
- link torso_link: mass 9.14397 -> 9.14489; geometry collision box size=0.16 0.2 0.25; visual box size=0.0453 0.0248 0.0358
Joints:
- joint left_ankle_roll: limit lower=-0.349066 upper=0.349066 effort=80.4 velocity=30.4781 -> lower=-0.349066 upper=0.349066 effort=84 velocity=29.1719
- joint right_ankle_roll: limit lower=-0.349066 upper=0.349066 effort=80.4 velocity=30.4781 -> lower=-0.349066 upper=0.349066 effort=84 velocity=29.1719

File: description/urdf/marvin_bot_covers.urdf (robot description, URDF)
Before this commit: robot marvin_bot, 28 links, 27 joints
Links:
- link left_ankle_link: mass 0.08558 -> 0.04888
- link left_foot_link: mass 0.57162 -> 0.43152
- link left_forearm_link: mass 0.54587 -> 0.54407
- link left_hip_pitch_link: mass 1.54966 -> 1.53913
- link left_hip_roll_link: mass 1.8617 -> 1.96168; geometry visual cylinder length=0.0132 radius=0.047; visual cylinder length=0.0425 radius=0.06
- link left_shin_link: mass 2.83858 -> 2.95671; geometry collision box size=0.104 0.09 0.097; collision box size=0.11 0.09 0.105
- link left_shoulder_pitch_link: mass 1.13716 -> 1.17592
- link left_shoulder_roll_link: mass 0.83212 -> 0.83559
- link left_thigh_link: mass 2.03853 -> 2.06227; geometry collision box size=0.09 0.09 0.16; visual box size=0.02 0.08 0.06
- link left_upper_arm_link: mass 0.88874 -> 0.90423
- link neck_link: mass 0.19965 -> 0.15145
- link pelvis: mass 5.35506 -> 6.42004; geometry collision box size=0.09 0.13 0.13; collision box size=0.09 0.13 0.13
- link right_ankle_link: mass 0.08558 -> 0.04888
- link right_foot_link: mass 0.57162 -> 0.43152
- link right_forearm_link: mass 0.54587 -> 0.54407
- link right_hip_pitch_link: mass 1.54966 -> 1.53913
- link right_hip_roll_link: mass 1.8617 -> 1.96168; geometry visual cylinder length=0.0132 radius=0.047; visual cylinder length=0.0425 radius=0.06
- link right_shin_link: mass 2.83858 -> 2.95671; geometry collision box size=0.104 0.09 0.097; collision box size=0.11 0.09 0.105
- link right_shoulder_pitch_link: mass 1.13716 -> 1.17592
- link right_shoulder_roll_link: mass 0.83212 -> 0.83559
- link right_thigh_link: mass 2.03853 -> 2.06227; geometry collision box size=0.09 0.09 0.16; visual box size=0.02 0.08 0.06
- link right_upper_arm_link: mass 0.88874 -> 0.90423
- link torso_link: mass 9.61363 -> 9.59313; geometry collision box size=0.16 0.2 0.25; visual box size=0.0453 0.0248 0.0358
Joints:
- joint left_ankle_roll: limit lower=-0.349066 upper=0.349066 effort=80.4 velocity=30.4781 -> lower=-0.349066 upper=0.349066 effort=84 velocity=29.1719
- joint right_ankle_roll: limit lower=-0.349066 upper=0.349066 effort=80.4 velocity=30.4781 -> lower=-0.349066 upper=0.349066 effort=84 velocity=29.1719

Commit message: CAD: RS03/RS06 on front rings, crossed-roller bearings, zero pins; aluminium load path
RobStride's drawings show the RS03 and RS06 are tapped only in ears at their
output end; the CAD bolted all 15 of them through their rear faces. Each now
hangs from a ring on its ears (cad/mounts.py: front_ring, hub, cage), the
ankle motors bolt straight to the shin plates, and the hip yaw motor moves
onto the thigh.

- RA6008 crossed-roller bearings at the hip yaw, the waist and in a carrier
  on each hip roll RS04's front face; the hip roll yoke's rear bearing set
  is gone
- stop pins in arc grooves (hard stops) and zero holes at nine joints
- the printed arm, neck, head-frame, wrist, hand-mount, battery-shelf and
  computer-plate parts are flat 7075 plates; the pelvis box and the printed
  chest and thigh shells under the covers are gone
- every metal part at SF 2.2 or better in cad/fea.py (pelvis at a 6 mm mesh)
- 42.29 kg bare, 43.24 kg with covers: tools/check_description.py still
  fails the 42 kg limit with covers until the next lightening round

Co-Authored-By: Claude Opus 5.5 <noreply@anthropic.com>

File: description/urdf/marvin_bot.urdf (robot description, URDF)
Before this commit: robot marvin_bot, 28 links, 27 joints
Links:
- link head_link: mass 0.36741 -> 0.40558; geometry collision box size=0.16 0.142 0.158; visual mesh filename=../meshes/head_camera.stl
- link left_forearm_link: mass 0.51981 -> 0.5592; geometry collision box size=0.07 0.07 0.17; visual box size=0.02 0.06 0.05
- link left_hip_pitch_link: mass 1.50236 -> 0.55044; geometry visual mesh filename=../meshes/left_hip_pitch_back.stl; visual mesh filename=../meshes/left_hip_pitch_bearing.stl
- link left_hip_roll_link: mass 1.96168 -> 1.86517; geometry visual cylinder length=0.0132 radius=0.047; visual cylinder length=0.0425 radius=0.06
- link left_palm_link: mass 0.41829 -> 0.44391; geometry collision box size=0.05 0.11 0.16; visual mesh filename=../meshes/left_hand.stl
- link left_shin_link: mass 2.89625 -> 2.73597; geometry collision box size=0.104 0.09 0.097; collision box size=0.11 0.09 0.105
- link left_shoulder_pitch_link: mass 1.16922 -> 1.02507; geometry visual cylinder length=0.0125 radius=0.039; visual cylinder length=0.0441 radius=0.05
- link left_shoulder_roll_link: mass 0.83559 -> 1.07479; geometry visual cylinder length=0.014 radius=0.035; visual cylinder length=0.0365 radius=0.0425
- link left_thigh_link: mass 2.02313 -> 3.18209; geometry collision box size=0.09 0.09 0.16; visual box size=0.02 0.08 0.06
- link left_upper_arm_link: mass 0.88431 -> 0.8644; geometry collision box size=0.08 0.08 0.14; visual cylinder length=0.014 radius=0.035
- link left_wrist_link: mass 0.11534 -> 0.11902; geometry collision box size=0.035 0.05 0.05; visual box size=0.0248 0.0358 0.0453
- link neck_link: mass 0.11085 -> 0.13365; geometry visual box size=0.0248 0.0358 0.0453; visual mesh filename=../meshes/neck_bracket.stl
- link pelvis: mass 6.38544 -> 6.85842; geometry collision box size=0.09 0.13 0.13; collision box size=0.09 0.13 0.13
- link right_forearm_link: mass 0.51981 -> 0.5592; geometry collision box size=0.07 0.07 0.17; visual box size=0.02 0.06 0.05
- link right_hip_pitch_link: mass 1.50236 -> 0.55044; geometry visual mesh filename=../meshes/right_hip_pitch_back.stl; visual mesh filename=../meshes/right_hip_pitch_bearing.stl
- link right_hip_roll_link: mass 1.96168 -> 1.86517; geometry visual cylinder length=0.0132 radius=0.047; visual cylinder length=0.0425 radius=0.06
- link right_palm_link: mass 0.41829 -> 0.44391; geometry collision box size=0.05 0.11 0.16; visual mesh filename=../meshes/right_hand.stl
- link right_shin_link: mass 2.89625 -> 2.73597; geometry collision box size=0.104 0.09 0.097; collision box size=0.11 0.09 0.105
- link right_shoulder_pitch_link: mass 1.16922 -> 1.02507; geometry visual cylinder length=0.0125 radius=0.039; visual cylinder length=0.0441 radius=0.05
- link right_shoulder_roll_link: mass 0.83559 -> 1.07479; geometry visual cylinder length=0.014 radius=0.035; visual cylinder length=0.0365 radius=0.0425
- link right_thigh_link: mass 2.02313 -> 3.18209; geometry collision box size=0.09 0.09 0.16; visual box size=0.02 0.08 0.06
- link right_upper_arm_link: mass 0.88431 -> 0.8644; geometry collision box size=0.08 0.08 0.14; visual cylinder length=0.014 radius=0.035
- link right_wrist_link: mass 0.11534 -> 0.11902; geometry collision box size=0.035 0.05 0.05; visual box size=0.0248 0.0358 0.0453
- link torso_link: mass 9.14489 -> 9.12885; geometry collision box size=0.16 0.2 0.25; visual box size=0.0453 0.0248 0.0358

File: description/urdf/marvin_bot_covers.urdf (robot description, URDF)
Before this commit: robot marvin_bot, 28 links, 27 joints
Links:
- link head_link: mass 0.36741 -> 0.40558; geometry collision box size=0.16 0.142 0.158; visual mesh filename=../meshes/head_camera.stl
- link left_forearm_link: mass 0.54407 -> 0.58366; geometry collision box size=0.07 0.07 0.17; visual box size=0.02 0.06 0.05
- link left_hip_pitch_link: mass 1.53913 -> 0.56557; geometry visual mesh filename=../meshes/left_hip_pitch_back.stl; visual mesh filename=../meshes/left_hip_pitch_bearing.stl
- link left_hip_roll_link: mass 1.96168 -> 1.86517; geometry visual cylinder length=0.0132 radius=0.047; visual cylinder length=0.0425 radius=0.06
- link left_palm_link: mass 0.41829 -> 0.44391; geometry collision box size=0.05 0.11 0.16; visual mesh filename=../meshes/left_hand.stl
- link left_shin_link: mass 2.95671 -> 2.79599; geometry collision box size=0.104 0.09 0.097; collision box size=0.11 0.09 0.105
- link left_shoulder_pitch_link: mass 1.17592 -> 1.03293; geometry visual cylinder length=0.0125 radius=0.039; visual cylinder length=0.0441 radius=0.05
- link left_shoulder_roll_link: mass 0.83559 -> 1.07479; geometry visual cylinder length=0.014 radius=0.035; visual cylinder length=0.0365 radius=0.0425
- link left_thigh_link: mass 2.06227 -> 3.24877; geometry collision box size=0.09 0.09 0.16; visual box size=0.02 0.08 0.06
- link left_upper_arm_link: mass 0.90423 -> 0.88377; geometry collision box size=0.08 0.08 0.14; visual cylinder length=0.014 radius=0.035
- link left_wrist_link: mass 0.11534 -> 0.11902; geometry collision box size=0.035 0.05 0.05; visual box size=0.0248 0.0358 0.0453
- link neck_link: mass 0.15145 -> 0.17425; geometry visual box size=0.0248 0.0358 0.0453; visual mesh filename=../meshes/neck_bracket.stl
- link pelvis: mass 6.42004 -> 6.89327; geometry collision box size=0.09 0.13 0.13; collision box size=0.09 0.13 0.13
- link right_forearm_link: mass 0.54407 -> 0.58366; geometry collision box size=0.07 0.07 0.17; visual box size=0.02 0.06 0.05
- link right_hip_pitch_link: mass 1.53913 -> 0.56557; geometry visual mesh filename=../meshes/right_hip_pitch_back.stl; visual mesh filename=../meshes/right_hip_pitch_bearing.stl
- link right_hip_roll_link: mass 1.96168 -> 1.86517; geometry visual cylinder length=0.0132 radius=0.047; visual cylinder length=0.0425 radius=0.06
- link right_palm_link: mass 0.41829 -> 0.44391; geometry collision box size=0.05 0.11 0.16; visual mesh filename=../meshes/right_hand.stl
- link right_shin_link: mass 2.95671 -> 2.79599; geometry collision box size=0.104 0.09 0.097; collision box size=0.11 0.09 0.105
- link right_shoulder_pitch_link: mass 1.17592 -> 1.03293; geometry visual cylinder length=0.0125 radius=0.039; visual cylinder length=0.0441 radius=0.05
- link right_shoulder_roll_link: mass 0.83559 -> 1.07479; geometry visual cylinder length=0.014 radius=0.035; visual cylinder length=0.0365 radius=0.0425
- link right_thigh_link: mass 2.06227 -> 3.24877; geometry collision box size=0.09 0.09 0.16; visual box size=0.02 0.08 0.06
- link right_upper_arm_link: mass 0.90423 -> 0.88377; geometry collision box size=0.08 0.08 0.14; visual cylinder length=0.014 radius=0.035
- link right_wrist_link: mass 0.11534 -> 0.11902; geometry collision box size=0.035 0.05 0.05; visual box size=0.0248 0.0358 0.0453
- link torso_link: mass 9.59313 -> 9.57935; geometry collision box size=0.16 0.2 0.25; visual box size=0.0453 0.0248 0.0358
