Commit message: CAD: lightened to 41.95 kg with covers, every metal part at SF 2.3 or better
- the pelvis box and rear gussets out (10 mm back plate instead), plates at
  SF 4 and up thinned or pocketed, the printed shells under the covers gone
- covers 1.0 mm, head shell 1.8 mm, TPU soles 3 mm
- cad/mounts.py: output_windows; thin rings pocketed only inside their screw
  circle; cad/fea.py checks cage strips through FEA-only bonded solids
- 41.16 kg bare, 41.95 kg with covers: tools/check_all.sh passes

Co-Authored-By: Claude Opus 5.5 <noreply@anthropic.com>

File: description/urdf/marvin_bot.urdf (robot description, URDF)
Before this commit: robot marvin_bot, 28 links, 27 joints
Links:
- link head_link: mass 0.40558 -> 0.35465
- link left_foot_link: mass 0.4149 -> 0.39163
- link left_forearm_link: mass 0.5592 -> 0.52858
- link left_hip_pitch_link: mass 0.55044 -> 0.42311
- link left_hip_roll_link: mass 1.86517 -> 1.83371
- link left_shin_link: mass 2.73597 -> 2.72405
- link left_shoulder_pitch_link: mass 1.02507 -> 1.02395
- link left_shoulder_roll_link: mass 1.07479 -> 1.02134
- link left_thigh_link: mass 3.18209 -> 3.14779
- link neck_link: mass 0.13365 -> 0.12519
- link pelvis: mass 6.85842 -> 6.63751; geometry collision box size=0.09 0.13 0.13; collision box size=0.09 0.13 0.13
- link right_foot_link: mass 0.4149 -> 0.39163
- link right_forearm_link: mass 0.5592 -> 0.52858
- link right_hip_pitch_link: mass 0.55044 -> 0.42311
- link right_hip_roll_link: mass 1.86517 -> 1.83371
- link right_shin_link: mass 2.73597 -> 2.72405
- link right_shoulder_pitch_link: mass 1.02507 -> 1.02395
- link right_shoulder_roll_link: mass 1.07479 -> 1.02134
- link right_thigh_link: mass 3.18209 -> 3.14779
- link torso_link: mass 9.12885 -> 8.9038

File: description/urdf/marvin_bot_covers.urdf (robot description, URDF)
Before this commit: robot marvin_bot, 28 links, 27 joints
Links:
- link head_link: mass 0.40558 -> 0.35465
- link left_foot_link: mass 0.43152 -> 0.40524
- link left_forearm_link: mass 0.58366 -> 0.54876
- link left_hip_pitch_link: mass 0.56557 -> 0.43579
- link left_hip_roll_link: mass 1.86517 -> 1.83371
- link left_shin_link: mass 2.79599 -> 2.774
- link left_shoulder_pitch_link: mass 1.03293 -> 1.03051
- link left_shoulder_roll_link: mass 1.07479 -> 1.02134
- link left_thigh_link: mass 3.24877 -> 3.20305
- link left_upper_arm_link: mass 0.88377 -> 0.88051
- link neck_link: mass 0.17425 -> 0.16579
- link pelvis: mass 6.89327 -> 6.66532; geometry collision box size=0.09 0.13 0.13; collision box size=0.09 0.13 0.13
- link right_foot_link: mass 0.43152 -> 0.40524
- link right_forearm_link: mass 0.58366 -> 0.54876
- link right_hip_pitch_link: mass 0.56557 -> 0.43579
- link right_hip_roll_link: mass 1.86517 -> 1.83371
- link right_shin_link: mass 2.79599 -> 2.774
- link right_shoulder_pitch_link: mass 1.03293 -> 1.03051
- link right_shoulder_roll_link: mass 1.07479 -> 1.02134
- link right_thigh_link: mass 3.24877 -> 3.20305
- link right_upper_arm_link: mass 0.88377 -> 0.88051
- link torso_link: mass 9.57935 -> 9.27772

Commit message: Harness clip points, faceted torso shell, shells refined to the new frame; docs synced
- Harness clips in the parts: push-in mount holes on solid pads (clip_spot), printed
  TPU edge clips for thick plates (cad/clips.py), a P-clip at the shoulder flange;
  CLIPS checked against cad_model.yaml.
- Torso shell faceted (alternating octagon sections, hulled), shoulder chamfers and a
  front bevel that clears the shoulder roll bracket; flat-shaded in renders.
- Grilles over the arm motors; room for each harness loop over the arc between its
  clip holes, on the rear arc at the knee (it had notched the thigh shell).
- 41.17 kg bare, 41.99 kg with shells; cad.covers --check finds no contacts.
- README, decisions, roadmap, wiring doc, the site's home page and guide pages 00 and
  08 updated (build123d frame, front rings, bearings, clips, shells); README render.

Co-Authored-By: Claude Opus 5.5 <noreply@anthropic.com>

File: description/urdf/marvin_bot.urdf (robot description, URDF)
Before this commit: robot marvin_bot, 28 links, 27 joints
Links:
- link left_forearm_link: mass 0.52858 -> 0.52081
- link left_hip_pitch_link: mass 0.42311 -> 0.42525; geometry visual mesh filename=../meshes/left_hip_pitch_back.stl; visual mesh filename=../meshes/left_hip_pitch_bearing.stl
- link left_hip_roll_link: mass 1.83371 -> 1.84062
- link left_shin_link: mass 2.72405 -> 2.72775
- link left_shoulder_roll_link: mass 1.02134 -> 1.00728; geometry visual cylinder length=0.014 radius=0.035; visual cylinder length=0.0365 radius=0.0425
- link left_thigh_link: mass 3.14779 -> 3.15606
- link left_upper_arm_link: mass 0.8644 -> 0.86196
- link left_wrist_link: mass 0.11902 -> 0.11874
- link neck_link: mass 0.12519 -> 0.12495
- link pelvis: mass 6.63751 -> 6.64042; geometry collision box size=0.09 0.13 0.13; collision box size=0.09 0.13 0.13
- link right_forearm_link: mass 0.52858 -> 0.52081
- link right_hip_pitch_link: mass 0.42311 -> 0.42525; geometry visual mesh filename=../meshes/right_hip_pitch_back.stl; visual mesh filename=../meshes/right_hip_pitch_bearing.stl
- link right_hip_roll_link: mass 1.83371 -> 1.84062
- link right_shin_link: mass 2.72405 -> 2.72775
- link right_shoulder_roll_link: mass 1.02134 -> 1.00728; geometry visual cylinder length=0.014 radius=0.035; visual cylinder length=0.0365 radius=0.0425
- link right_thigh_link: mass 3.14779 -> 3.15606
- link right_upper_arm_link: mass 0.8644 -> 0.86196
- link right_wrist_link: mass 0.11902 -> 0.11874
- link torso_link: mass 8.9038 -> 8.91884; geometry collision box size=0.16 0.2 0.25; visual box size=0.0453 0.0248 0.0358

File: description/urdf/marvin_bot_covers.urdf (robot description, URDF)
Before this commit: robot marvin_bot, 28 links, 27 joints
Links:
- link left_forearm_link: mass 0.54876 -> 0.53861
- link left_hip_pitch_link: mass 0.43579 -> 0.43793; geometry visual mesh filename=../meshes/left_hip_pitch_back.stl; visual mesh filename=../meshes/left_hip_pitch_bearing.stl
- link left_hip_roll_link: mass 1.83371 -> 1.84062
- link left_shin_link: mass 2.774 -> 2.7777
- link left_shoulder_roll_link: mass 1.02134 -> 1.00728; geometry visual cylinder length=0.014 radius=0.035; visual cylinder length=0.0365 radius=0.0425
- link left_thigh_link: mass 3.20305 -> 3.21132
- link left_upper_arm_link: mass 0.88051 -> 0.87666
- link left_wrist_link: mass 0.11902 -> 0.11874
- link neck_link: mass 0.16579 -> 0.16555
- link pelvis: mass 6.66532 -> 6.66823; geometry collision box size=0.09 0.13 0.13; collision box size=0.09 0.13 0.13
- link right_forearm_link: mass 0.54876 -> 0.53861
- link right_hip_pitch_link: mass 0.43579 -> 0.43793; geometry visual mesh filename=../meshes/right_hip_pitch_back.stl; visual mesh filename=../meshes/right_hip_pitch_bearing.stl
- link right_hip_roll_link: mass 1.83371 -> 1.84062
- link right_shin_link: mass 2.774 -> 2.7777
- link right_shoulder_roll_link: mass 1.02134 -> 1.00728; geometry visual cylinder length=0.014 radius=0.035; visual cylinder length=0.0365 radius=0.0425
- link right_thigh_link: mass 3.20305 -> 3.21132
- link right_upper_arm_link: mass 0.88051 -> 0.87666
- link right_wrist_link: mass 0.11902 -> 0.11874
- link torso_link: mass 9.27772 -> 9.33108; geometry collision box size=0.16 0.2 0.25; visual box size=0.0453 0.0248 0.0358
